File: kicad/audio.kicad_sch (KiCad schematic)
At the start: 12 parts, among them J3 AudioJack4_Ground_SwitchTR1, U9 CS43131-CNZR, Y4 22.5792MHz

Commit message: changes
Parts:
- J3: value AudioJack4_Ground_SwitchTR1 -> SHOU HAN PJ-342
Changed lines of the file:
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@@
 			)
 		)
-		(property "Value" "AudioJack4_Ground_SwitchTR1"
+		(property "Value" "SHOU HAN PJ-342"
 			(at 20.8915 63.5 0)
 			(show_name no)
