File: kicad/audio.kicad_sch (KiCad schematic)
At the start: 12 parts, among them J3 SHOU HAN PJ-342, U9 CS43131-CNZR

Commit message: changes to audio sheet
Connections:
- net GND: now also U9.41 (EP)
Changed lines of the file:
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@@
+	)
+	(junction
+		(at 140.97 127)
+		(diameter 0)
+		(color 0 0 0 0)
 	)
 	(junction
@@
 	(wire
 		(pts
+			(xy 138.43 127) (xy 140.97 127)
+		)
+		(stroke
+			(width 0)
+			(type default)
+		)
+	)
+	(wire
+		(pts
 			(xy 199.39 54.61) (xy 199.39 55.88)
 		)
@@
 		)
 		(stroke
+			(width 0)
+			(type default)
+		)
+	)
+	(wire
+		(pts
+			(xy 138.43 125.73) (xy 138.43 127)
+		)
+		(stroke

Commit message: almost done!
Parts:
- removed J3: SHOU HAN PJ-342, symbol Connector_Audio:AudioJack4_Ground_SwitchTR1
- added J4: AudioJack3_Ground_SwitchTR, Connector_Audio:Jack_3.5mm_PJ31060-I_Horizontal, symbol Connector_Audio:AudioJack3_Ground_SwitchTR
- C34, C35, C36, C37, C38, C39, C40, C41, C42: footprint (none) -> Capacitor_SMD:C_0603_1608Metric
Connections:
- net GND: now also J4.G, J4.S
- net at U9.14 (HPOUTA): now also J4.T
- net at U9.16 (HPOUTB): now also J4.R
- net at U9.22 (HP_DETECT): now also J4.TN
- no-connect marks 8 -> 7
Changed lines of the file:
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@@
-	)
-	(no_connect
-		(at 201.93 114.3)
 	)
 	(no_connect
@@
 	)
 	(no_connect
-		(at 201.93 121.92)
+		(at 209.55 121.92)
 	)
 	(no_connect
@@
 	(wire
 		(pts
-			(xy 201.93 116.84) (xy 199.39 116.84)
+			(xy 209.55 116.84) (xy 199.39 116.84)
 		)
 		(stroke
@@
 	(wire
 		(pts
-			(xy 207.01 132.08) (xy 207.01 133.35)
+			(xy 214.63 132.08) (xy 214.63 133.35)
 		)
 		(stroke
@@
 	(wire
 		(pts
-			(xy 190.5 119.38) (xy 201.93 119.38)
+			(xy 190.5 119.38) (xy 209.55 119.38)
 		)
 		(stroke
@@
 	(wire
 		(pts
-			(xy 189.23 124.46) (xy 201.93 124.46)
+			(xy 189.23 124.46) (xy 209.55 124.46)
 		)
 		(stroke
@@
 	(wire
 		(pts
-			(xy 187.96 127) (xy 201.93 127)
+			(xy 187.96 127) (xy 209.55 127)
 		)
 		(stroke
@@
 	)
 	(symbol
+		(lib_id "Connector_Audio:AudioJack3_Ground_SwitchTR")
+		(at 214.63 119.38 0)
+		(mirror y)
+		(unit 1)
+		(body_style 1)
+		(exclude_from_sim no)
+		(in_bom yes)
+		(on_board yes)
+		(in_pos_files yes)
+		(dnp no)
+		(property "Reference" "J4"
+			(at 216.535 110.49 0)
+			(show_name no)
+			(do_not_autoplace no)
+			(effects
+				(font
+					(size 1.27 1.27)
+				)
+			)
+		)
+		(property "Value" "AudioJack3_Ground_SwitchTR"
+			(at 216.535 113.03 0)
+			(show_name no)
+			(do_not_autoplace no)
+			(effects
+				(font
+					(size 1.27 1.27)
+				)
+			)
+		)
+		(property "Footprint" "Connector_Audio:Jack_3.5mm_PJ31060-I_Horizontal"
+			(at 214.63 119.38 0)
+			(hide yes)
+			(show_name no)
+			(do_not_autoplace no)
+			(effects
+				(font
+					(size 1.27 1.27)
+				)
+			)
+		)
+		(property "Datasheet" ""
+			(at 214.63 119.38 0)
+			(hide yes)
+			(show_name no)
+			(do_not_autoplace no)
+			(effects
+				(font
+					(size 1.27 1.27)
+				)
+			)
+		)
+		(property "Description" "Audio Jack, 3 Poles (Stereo / TRS), Grounded Sleeve, Switched TR Poles (Normalling)"
+			(at 214.63 119.38 0)
+			(hide yes)
+			(show_name no)
+			(do_not_autoplace no)
+			(effects
+				(font
+					(size 1.27 1.27)
+				)
+			)
+		)
+		(pin "TN"
+		)
+		(pin "T"
+		)
+		(pin "S"
+		)
+		(pin "RN"
+		)
+		(pin "G"
+		)
+		(pin "R"
+		)
+		(instances
+			(project "MP3player"
+				(path "/c86fdb70-ebb0-4c87-946f-42a0fbefb388/8ec0c330-8240-4e36-aed2-8b84a8e7f410"
+					(reference "J4")
+					(unit 1)
+				)
+			)
+		)
+	)
+	(symbol
 		(lib_id "power:GND")
 		(at 175.26 74.93 0)
@@
 			)
 		)
-		(property "Footprint" ""
+		(property "Footprint" "Capacitor_SMD:C_0603_1608Metric"
 			(at 199.39 58.42 0)
 			(hide yes)
@@
 			)
 		)
-		(property "Footprint" ""
+		(property "Footprint" "Capacitor_SMD:C_0603_1608Metric"
 			(at 186.69 58.42 0)
 			(hide yes)
@@
 			)
 		)
-		(property "Footprint" ""
+		(property "Footprint" "Capacitor_SMD:C_0603_1608Metric"
 			(at 109.22 59.69 0)
 			(hide yes)
@@
 			)
 		)
-		(property "Footprint" ""
+		(property "Footprint" "Capacitor_SMD:C_0603_1608Metric"
 			(at 160.02 62.23 0)
 			(hide yes)
@@
 			)
 		)
-		(property "Footprint" ""
+		(property "Footprint" "Capacitor_SMD:C_0603_1608Metric"
 			(at 180.34 69.85 0)
 			(hide yes)
@@
 			)
 		)
-		(property "Footprint" ""
+		(property "Footprint" "Capacitor_SMD:C_0603_1608Metric"
 			(at 160.02 69.85 0)
 			(hide yes)
@@
 	(symbol
 		(lib_id "power:GND")
-		(at 207.01 133.35 0)
+		(at 214.63 133.35 0)
 		(unit 1)
 		(body_style 1)
@@
 		(fields_autoplaced yes)
 		(property "Reference" "#PWR048"
-			(at 207.01 139.7 0)
+			(at 214.63 139.7 0)
 			(hide yes)
 			(show_name no)
@@
 		)
 		(property "Value" "GND"
-			(at 207.01 138.43 0)
+			(at 214.63 138.43 0)
 			(show_name no)
 			(do_not_autoplace no)
@@
 		)
 		(property "Footprint" ""
-			(at 207.01 133.35 0)
+			(at 214.63 133.35 0)
 			(hide yes)
 			(show_name no)
@@
 		)
 		(property "Datasheet" ""
-			(at 207.01 133.35 0)
+			(at 214.63 133.35 0)
 			(hide yes)
 			(show_name no)
@@
 		)
 		(property "Description" "Power symbol creates a global label with name \"GND\" , ground"
-			(at 207.01 133.35 0)
+			(at 214.63 133.35 0)
 			(hide yes)
 			(show_name no)
@@
 			)
 		)
-		(property "Footprint" ""
+		(property "Footprint" "Capacitor_SMD:C_0603_1608Metric"
 			(at 170.18 69.85 0)
 			(hide yes)
@@
 			)
 		)
-		(property "Footprint" ""
+		(property "Footprint" "Capacitor_SMD:C_0603_1608Metric"
 			(at 97.79 59.69 0)
 			(hide yes)
@@
 			)
 		)
-		(property "Footprint" ""
+		(property "Footprint" "Capacitor_SMD:C_0603_1608Metric"
 			(at 160.02 80.01 0)
 			(hide yes)
@@
 					(unit 1)
 				)
-			)
-		)
-	)
-	(symbol
-		(lib_id "Connector_Audio:AudioJack4_Ground_SwitchTR1")
-		(at 207.01 119.38 0)
-		(mirror y)
-		(unit 1)
-		(body_style 1)
-		(exclude_from_sim no)
-		(in_bom yes)
-		(on_board yes)
-		(in_pos_files yes)
-		(dnp no)
-		(property "Reference" "J3"
-			(at 210.2485 107.95 0)
-			(show_name no)
-			(do_not_autoplace no)
-			(effects
-				(font
-					(size 1.27 1.27)
-				)
-			)
-		)
-		(property "Value" "SHOU HAN PJ-342"
-			(at 210.2485 110.49 0)
-			(show_name no)
-			(do_not_autoplace no)
-			(effects
-				(font
-					(size 1.27 1.27)
-				)
-			)
-		)
-		(property "Footprint" ""
-			(at 208.28 119.38 0)
-			(hide yes)
-			(show_name no)
-			(do_not_autoplace no)
-			(effects
-				(font
-					(size 1.27 1.27)
-				)
-			)
-		)
-		(property "Datasheet" ""
-			(at 208.28 119.38 0)
-			(hide yes)
-			(show_name no)
-			(do_not_autoplace no)
-			(effects
-				(font
-					(size 1.27 1.27)
-				)
-			)
-		)
-		(property "Description" "Audio Jack, 4 Poles (Stereo / TRRS), Grounded Sleeve, Switched TR1 Poles (Normalling)"
-			(at 207.01 119.38 0)
-			(hide yes)
-			(show_name no)
-			(do_not_autoplace no)
-			(effects
-				(font
-					(size 1.27 1.27)
-				)
-			)
-		)
-		(pin "S"
-		)
-		(pin "TN"
-		)
-		(pin "R2"
-		)
-		(pin "T"
-		)
-		(pin "G"
-		)
-		(pin "R1N"
-		)
-		(pin "R1"
-		)
-		(instances
-			(project "MP3player"
-				(path "/c86fdb70-ebb0-4c87-946f-42a0fbefb388/8ec0c330-8240-4e36-aed2-8b84a8e7f410"
-					(reference "J3")
-					(unit 1)
-				)

Commit message: general changes
Parts:
- TP3: footprint (none) -> TestPoint:TestPoint_Pad_D1.5mm
- U9: footprint easyeda2kicad:TQFN-40_L5.0-W5.0-P0.40-TL-EP3.5 -> Package_DFN_QFN:TQFN-40-1EP_5x5mm_P0.4mm_EP3.5x3.5mm
Connections:
- net GND: now also J4.1, J4.2; no longer J4.G, J4.S
- net at U9.14 (HPOUTA): now also J4.4; no longer J4.T
- net at U9.16 (HPOUTB): now also J4.3; no longer J4.R
- net at U9.22 (HP_DETECT): now also J4.6; no longer J4.TN
Changed lines of the file:
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@@
 			)
 		)
-		(property "Footprint" "easyeda2kicad:TQFN-40_L5.0-W5.0-P0.40-TL-EP3.5"
+		(property "Footprint" "Package_DFN_QFN:TQFN-40-1EP_5x5mm_P0.4mm_EP3.5x3.5mm"
 			(at 143.51 151.13 0)
 			(hide yes)
@@
 			)
 		)
-		(pin "TN"
-		)
-		(pin "T"
-		)
-		(pin "S"
-		)
-		(pin "RN"
-		)
-		(pin "G"
-		)
-		(pin "R"
+		(pin "6"
+		)
+		(pin "2"
+		)
+		(pin "1"
+		)
+		(pin "3"
+		)
+		(pin "4"
+		)
+		(pin "5"
 		)
 		(instances
@@
 			)
 		)
-		(property "Footprint" ""
+		(property "Footprint" "TestPoint:TestPoint_Pad_D1.5mm"
 			(at 127 57.15 0)
 			(hide yes)
