File: kicad/radio.kicad_sch (KiCad schematic)
At the start: 1 part, among them U12 Si4735-D60-GU

Commit message: updates
Parts:
- added C131: 22nF, symbol Device:C_Small
- added C132, C133: 1nF, symbol Device:C_Small
- added C134, C135: 22pF, symbol Device:C_Small
- added C136: 2-5pF, symbol Device:C_Small
- added C48, C49: 0.1uF, symbol Device:C_Small
- added L3: 180-450uH, Inductor_SMD:L_2512_6332Metric, symbol Device:L_Ferrite
- added R26: 600, symbol Device:R_Small_US
- added R27, R28: 2k, symbol Device:R_Small_US
- added Y3: 32.768KHz, symbol Device:Crystal
- renumbered U12 to U10
Connections:
- net 3.3V: now also U10.20 (VD), U10.21 (VA), C131.1, C48.1, C49.1
- net GND: now also C134.2, C135.2, C136.2, C48.2, C49.2
- net at U10.1 (DOUT): now also R26.1
- net at U10.12 (AMI): now also C133.1
- net RST: now reaches U10.15 (~{RST})
- net SEN: now reaches U10.16 (~{SEN})
- net SCLK: now reaches U10.17 (SCLK)
- net SDIO: now reaches U10.18 (SDIO)
- net at U10.19 (RCLK): now also C135.1, Y3.1
- net at U10.2 (DFS): now also R27.1
- net at U10.22 (DBYP): now also C131.2
- net ROUT: now reaches U10.23 (ROUT/[DOUT])
- net LOUT: now reaches U10.24 (LOUT/[DFS])
- net at U10.3 (GPO3/[DCLK]): now also R28.2
- net GPO2/INT: now reaches U10.4 (GPO2/[~{INT}])
- net GPO1: now reaches U10.5 (GPO1)
- net at U10.8 (FMI): now also C132.1
- net at U10.9 (RFGND): now also L3.2
- new net: C134.1, R28.1, Y3.2
- new net DFS: C133.2, C136.1, L3.1, R27.2
- new net DOUT: R26.2
