File: kicad/sparkles.kicad_sch (KiCad schematic)
At the start: 160 parts

Commit message: almost done!
Parts:
- C100, C101, C102, C103, C104, C105, C106, C107, C108, C109, C110, C111, C112, C113, C114, C115, C116, C117, C118, C119, C120, C121, C122, C123, C124, C125, C126, C127, C128, C49, C50, C51, C52, C53, C54, C55, C56, C57, C58, C59, C60, C61, C62, C63, C64, C65, C66, C67, C68, C69, C70, C71, C72, C73, C74, C75, C76, C77, C78, C79, C80, C81, C82, C83, C84, C85, C86, C87, C88, C89, C90, C91, C92, C93, C94, C95, C96, C97, C98, C99: footprint (none) -> Capacitor_SMD:C_0603_1608Metric

Commit message: general changes
Parts:
- removed C100, C101, C102, C103, C104, C105, C106, C107, C108, C109, C110, C111, C112, C113, C114, C115, C116, C117, C118, C119, C120, C121, C122, C123, C124, C125, C126, C127, C128, C50, C51, C52, C53, C54, C55, C56, C58, C59, C60, C61, C62, C63, C64, C66, C67, C68, C69, C70, C71, C72, C74, C75, C76, C77, C78, C79, C80, C81, C82, C83, C84, C85, C86, C87, C88, C89, C90, C91, C92, C93, C94, C95, C96, C97, C98, C99: 0.1uF, Capacitor_SMD:C_0603_1608Metric, symbol Device:C_Small
- removed D10, D11, D13, D14, D15, D16, D17, D18, D19, D21, D22, D23, D24, D25, D26, D27, D29, D30, D31, D32, D33, D34, D35, D36, D37, D38, D39, D40, D41, D42, D43, D44, D45, D46, D47, D48, D49, D5, D50, D51, D52, D53, D54, D55, D56, D57, D58, D59, D6, D60, D61, D62, D63, D64, D65, D66, D67, D68, D69, D7, D70, D71, D72, D73, D74, D75, D76, D77, D78, D79, D8, D80, D81, D82, D83, D9: APA102-2020, LED_SMD:LED-APA102-2020, symbol LED:APA102-2020
- renumbered C57 to C50, C65 to C51, C73 to C52, D12 to D5, D20 to D6, D28 to D7
Connections:
- net CLKOUT: now also D7.2 (CKO)
- net DOUT: now also D7.3 (SDO)
- net GND: now reaches C49.2, C50.2, C51.2, C52.2, D4.6 (GND), D5.6 (GND), D6.6 (GND), D7.6 (GND)
