File: kicad/MP3player.kicad_pcb (KiCad board)
At the start: 2 copper layers, 50 x 70 mm, 259 parts, among them J1 USB_C_Receptacle_USB2.0_14P, J2 Conn_01x02, J3 Conn_01x05, J4 AudioJack3_Ground_SwitchTR, J6 SMA, J7 SMA, J8 Conn_01x08, SW1 SW_Push, SW10 SW_Push, SW11 SW_Push, SW12 SW_Push, SW13 SW_Push, SW14 SW_Push, SW15 SW_Push, SW16 SW_Push, SW17 SW_Push, SW2 SW_Push, SW3 SW_Push, SW4 SW_Push, SW5 SW_Push, SW6 SW_Push, SW7 SW_Push, SW8 SW_Push, SW9 SW_Push, U1 USBLC6-2SC6, U10 Si4735-D60-GU, U2 TLV70233_SOT23-5, U3 TPS7A4701xRGW, U4 STM32H743VIT6, U5 ISL29035, U6 LSM6DSL, U7 DS3231M, U8 BME680

Commit message: add images
Parts:
- moved C108 67.8 mm to (138.0, 151.0), turned to 180 degrees
- moved C116 64.4 mm to (142.0, 151.0), turned to 180 degrees
- moved C84 64.1 mm to (126.0, 151.0), turned to 180 degrees
- moved C124 62.5 mm to (146.0, 151.0), turned to 180 degrees
- moved C92 60.6 mm to (130.0, 151.0), turned to 180 degrees
- moved C60 60.5 mm to (114.0, 151.0), turned to 180 degrees
- moved C100 58.6 mm to (134.0, 151.0), turned to 180 degrees
- moved C68 56.8 mm to (118.0, 151.0), turned to 180 degrees
- moved C76 54.6 mm to (122.0, 151.0), turned to 180 degrees
- moved C52 50.7 mm to (110.0, 151.0), turned to 180 degrees
- moved C99 41.4 mm to (134.0, 145.0), turned to 180 degrees
- moved C107 39.3 mm to (138.0, 145.0), turned to 180 degrees
- moved C123 37.5 mm to (146.0, 145.0), turned to 180 degrees
- moved C115 37.1 mm to (142.0, 145.0), turned to 180 degrees
- moved D10 2.00 mm to (110.0, 162.0)
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
Commit message: general changes
Parts:
- removed BT1: CR2032, Battery:BatteryHolder_Keystone_3002_1x2032
- removed BT2: Battery_Cell, Battery:BatteryHolder_Keystone_3002_1x2032
- removed C100, C101, C102, C103, C104, C105, C106, C107, C108, C109, C110, C111, C112, C113, C114, C115, C116, C117, C118, C119, C120, C121, C122, C123, C124, C125, C126, C127, C128, C63, C64, C66, C67, C68, C69, C70, C71, C72, C74, C75, C76, C77, C78, C79, C80, C81, C82, C83, C84, C85, C86, C87, C88, C89, C90, C91, C92, C93, C94, C95, C96, C97, C98, C99: 0.1uF, Capacitor_SMD:C_0603_1608Metric
- removed C12, C9: 8pF, Capacitor_SMD:C_0603_1608Metric
- removed the C50 at (110.0, 139.0)
- removed the C51 at (110.0, 145.0)
- removed the C52 at (110.0, 151.0)
- removed the C53 at (59.8, 160.4)
- removed the C54 at (59.8, 162.9)
- removed the C55 at (59.8, 165.4)
- removed the C56 at (123.3, 198.3)
- removed the C58 at (114.0, 139.0)
- removed D11, D13, D14, D15, D16, D17, D18, D19, D21, D22, D23, D24, D25, D26, D27, D29, D30, D31, D32, D33, D34, D35, D36, D37, D38, D39, D40, D41, D42, D43, D44, D45, D46, D47, D48, D49, D50, D51, D52, D53, D54, D55, D56, D57, D58, D59, D60, D61, D62, D63, D64, D65, D66, D67, D68, D69, D70, D71, D72, D73, D74, D75, D76, D77, D78, D79, D80, D81, D82, D83: APA102-2020, LED_SMD:LED-APA102-2020
- removed the D5 at (110.0, 136.0)
- removed the D6 at (110.0, 142.0)
- removed the D7 at (110.0, 148.0)
- added J5: Micro_SD_Card_Det2, Connector_Card:microSD_HC_Hirose_DM3D-SF, F.Cu at (68.0, 72.8)
- added JP1: SolderJumper_3_Bridged12, Jumper:SolderJumper-3_P1.3mm_Bridged12_RoundedPad1.0x1.5mm, F.Cu at (55.5, 55.0)
- added L2: 2.2uH, Inductor_SMD:L_0805_2012Metric, F.Cu at (33.8, 62.6)
- added R1: 5.1k, Resistor_SMD:R_0603_1608Metric, F.Cu at (46.7, 84.7)
- added R10: 10k, Resistor_SMD:R_0603_1608Metric, F.Cu at (55.5, 58.5)
- added R11: 600, Resistor_SMD:R_0603_1608Metric, F.Cu at (44.5, 48.5)
- added R12: 10k, Resistor_SMD:R_0603_1608Metric, B.Cu at (52.5, 27.0)
- added R13: 10k, Resistor_SMD:R_0603_1608Metric, F.Cu at (27.0, 35.0)
- added R14: 10k, Resistor_SMD:R_0603_1608Metric, F.Cu at (-75.9, 50.5)
- added R15: 10k, Resistor_SMD:R_0603_1608Metric, F.Cu at (-75.9, 53.0)
- added R16: 10k, Resistor_SMD:R_0603_1608Metric, F.Cu at (-75.9, 55.5)
- added R17: 10k, Resistor_SMD:R_0603_1608Metric, B.Cu at (27.0, 45.5)
- added R18: 10k, Resistor_SMD:R_0603_1608Metric, B.Cu at (27.0, 53.5)
- added R19: 10k, Resistor_SMD:R_0603_1608Metric, B.Cu at (27.0, 61.5)
- added R2: 5.1k, Resistor_SMD:R_0603_1608Metric, F.Cu at (53.3, 84.8)
- added R20: 10k, Resistor_SMD:R_0603_1608Metric, F.Cu at (-63.9, 57.5)
- added R21: 1.5k, Resistor_SMD:R_0603_1608Metric, F.Cu at (40.0, 90.0)
- added R22: 1.5k, Resistor_SMD:R_0603_1608Metric, F.Cu at (37.0, 90.0)
- added R23: 1.1k, Resistor_SMD:R_0603_1608Metric, F.Cu at (32.4, 75.0)
- added R24: 11k, Resistor_SMD:R_0603_1608Metric, F.Cu at (42.8, 80.4)
- added R25: 1.1k, Resistor_SMD:R_0603_1608Metric, F.Cu at (34.0, 75.0)
- added R26: 5.11R, Resistor_SMD:R_0603_1608Metric, F.Cu at (32.8, 56.6)
- added R3: 22, Resistor_SMD:R_0603_1608Metric, F.Cu at (49.0, 83.9)
- added R4: 22, Resistor_SMD:R_0603_1608Metric, F.Cu at (51.0, 83.9)
- added R5: 10k, Resistor_SMD:R_0603_1608Metric, F.Cu at (-63.9, 45.5)
- added R6: 10k, Resistor_SMD:R_0603_1608Metric, B.Cu at (53.0, 34.5)
- added R7: 10k, Resistor_SMD:R_0603_1608Metric, B.Cu at (67.7, 64.8)
- added R8: 10k, Resistor_SMD:R_0603_1608Metric, B.Cu at (65.7, 64.8)
- added R9: 10k, Resistor_SMD:R_0603_1608Metric, F.Cu at (-63.9, 62.0)
- added TH1: 10k, Resistor_SMD:R_0603_1608Metric, F.Cu at (42.8, 78.5)
- added TP3: TestPoint, TestPoint:TestPoint_Pad_D1.5mm, F.Cu at (53.5, 80.0)
- added TP4: TestPoint, TestPoint:TestPoint_Pad_D1.5mm, F.Cu at (59.0, 52.0)
- added TP5: TestPoint, TestPoint:TestPoint_Pad_D1.5mm, F.Cu at (59.0, 48.5)
- added TP6: TestPoint, TestPoint:TestPoint_Pad_D1.5mm, F.Cu at (48.5, 46.0)
- added U11: BQ24090DGQ, Package_SO:HVSSOP-10-1EP_3x3mm_P0.5mm_EP1.83x1.89mm, F.Cu at (38.0, 79.0)
- added U12: TPS613222ADBV, Package_TO_SOT_SMD:SOT-23-5, F.Cu at (35.8, 59.6)
- added U9: CS43131-CNZR, Package_DFN_QFN:TQFN-40-1EP_5x5mm_P0.4mm_EP3.5x3.5mm, B.Cu at (60.7, 87.6)
- added Y1: 8MHz TXC AA08000002, Crystal:Crystal_SMD_5032-2Pin_5.0x3.2mm, B.Cu at (63.1, 44.7)
- C10, C17, C18, C19, C21, C27, C30, C32, C36, C37, C38, C39, C40, C41, C42, C49, D4, U4, U7: moved to B.Cu
- C11, C8: value 18pF -> 12pF; moved to B.Cu
- C50: renamed from C57; moved to B.Cu
- C51: renamed from C65; moved to B.Cu
- C52: renamed from C73; moved to B.Cu
- C54: renamed from C130; moved to B.Cu
- C55: renamed from C131; moved to B.Cu
- C56: renamed from C132; moved to B.Cu
- C57: renamed from C133; moved to B.Cu
- C58: renamed from C134; moved to B.Cu
- C59: value 0.1uF -> 1uF
- C60: value 0.1uF -> 4.7uF
- C61: value 0.1uF -> 22uF
- C62: value 0.1uF -> 120pF
- D1, D2, D3: footprint Package_TO_SOT_SMD:SOT-23-3 -> Package_TO_SOT_SMD:SOT-363_SC-70-6; moved to B.Cu
- D10: value APA102-2020 -> BAT54W; footprint LED_SMD:LED-APA102-2020 -> Package_TO_SOT_SMD:SOT-323_SC-70
- D5: renamed from D12; moved to B.Cu
- D6: renamed from D20; moved to B.Cu
- D7: renamed from D28; moved to B.Cu
- D8, D9: value APA102-2020 -> LED; footprint LED_SMD:LED-APA102-2020 -> LED_SMD:LED_0603_1608Metric
- J8: footprint Connector_PinHeader_2.54mm:PinHeader_1x08_P2.54mm_Vertical -> Connector_PinHeader_2.54mm:PinHeader_1x08_P2.54mm_Vertical_SMD_Pin1Right
- SW10, SW11, SW12, SW13, SW14, SW15, SW16, SW17, SW9: footprint Button_Switch_SMD:SW_Push_1P1T_NO_CK_KSC9xxJ -> Button_Switch_SMD:SW_Push_1P1T_NO_CK_KMR2
- moved H1 190.4 mm to (70.0, 29.9)
- moved H2 190.4 mm to (30.0, 29.9)
- moved H3 190.4 mm to (30.0, 89.9)
- moved H4 190.4 mm to (70.0, 89.9)
- moved J6 190.4 mm to (39.3, 29.5)
- moved J7 190.4 mm to (60.7, 29.5)
- moved C53 159.9 mm to (50.0, 34.5), turned to 180 degrees
- moved C27 152.4 mm to (46.5, 28.0), turned to 180 degrees
- moved C20 149.6 mm to (55.2, 34.1), turned to 90 degrees
- moved C47 143.4 mm to (56.0, 50.0), turned to 180 degrees
- moved C14 142.8 mm to (55.9, 45.4), turned to -90 degrees
- moved C21 142.7 mm to (39.4, 39.7), turned to 180 degrees
- moved C48 138.4 mm to (44.5, 53.0), turned to 180 degrees
- moved C8 135.9 mm to (63.1, 40.7), turned to 180 degrees
- moved C11 135.5 mm to (63.1, 48.7)
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- renumbered C129 to C53
Connections:
- net /Power/FORCE renamed /STM32 Core/PMM_FORCE
- net /Power/INIT renamed /STM32 Core/PMM_INIT
- net /Power/SCL renamed /STM32 Core/PWR_I2C_SCL
- net /Power/SDA renamed /STM32 Core/PWR_I2C_SDA
- net /Power/SHDN renamed /STM32 Core/PMM_SHDN
- net /Power/UART_RX renamed /STM32 Core/PMM_TX
- net /Power/UART_TX renamed /STM32 Core/PMM_RX
- C10 pad 1: /Microphone/3.3V -> +3.3V
- C10 pad 2: Net-(C10-Pad2) -> GND
- C14 pad 1: /Microphone/3.3V -> +3.3V
- C14 pad 2: Net-(C10-Pad2) -> GND
- C15 pad 1: /Microphone/3.3V -> +3.3V
- C15 pad 2: Net-(C10-Pad2) -> GND
- C17 pad 1: /Microphone/3.3V -> +3.3V
- C17 pad 2: Net-(C10-Pad2) -> GND
- C19 pad 1: Net-(BT1-+) -> +3.3V
- C20 pad 1: /Microphone/3.3V -> +3.3V
- C20 pad 2: Net-(C10-Pad2) -> GND
- C25 pad 1: /Microphone/3.3V -> +3.3V
- C26 pad 1: /Microphone/3.3V -> +3.3V
- C27 pad 1: /Microphone/3.3V -> +3.3V
- C28 pad 1: /Microphone/3.3V -> +3.3V
- C29 pad 1: /Microphone/3.3V -> +3.3V
- C3 pad 1: /Microphone/3.3V -> +3.3V
- C30 pad 1: /Microphone/3.3V -> +3.3V
- C31 pad 1: /Microphone/3.3V -> +3.3V
- C32 pad 1: Net-(BT2-+) -> +BATT
- C33 pad 1: /Microphone/3.3V -> +3.3V
- C4 pad 1: /Microphone/3.3V -> +3.3V
- C43 pad 1: /Microphone/3.3V -> +3.3V
- C44 pad 1: /Microphone/3.3V -> +3.3V
- C45 pad 1: /Microphone/3.3V -> +3.3V
- C47 pad 1: /Microphone/3.3V -> +3.3V
- C49 pad 2: Net-(D12-GND) -> GND
- C50 pad 2: Net-(D12-GND) -> GND
- C51 pad 2: Net-(D12-GND) -> GND
- C52 pad 2: Net-(D12-GND) -> GND
- C53 pad 1: /Microphone/3.3V -> +3.3V
- C59 pad 2: Net-(D14-GND) -> GND
- C60 pad 1: +5V -> +BATT
- C60 pad 2: Net-(D15-GND) -> GND
- C61 pad 2: Net-(D16-GND) -> GND
- C62 pad 1: +5V -> Net-(C62-Pad1)
- C62 pad 2: Net-(D17-GND) -> +5V
- D10 pad 1: +5V -> Net-(D10-A)
- D10 pad 2: Net-(D10-CKO) -> unconnected-(D10-NC-Pad2)
- D10 pad 3: Net-(D10-SDO) -> +5V
- D4 pad 6: Net-(D12-GND) -> GND
- D5 pad 6: Net-(D12-GND) -> GND
- D6 pad 6: Net-(D12-GND) -> GND
- D7 pad 2: Net-(D28-CKO) -> /LED Spectrum/CLKOUT
- D7 pad 3: Net-(D28-SDO) -> /LED Spectrum/DOUT
- D7 pad 6: Net-(D12-GND) -> GND
- D8 pad 1: +5V -> Net-(D8-K)
- D9 pad 1: +5V -> Net-(D9-K)
- FB1 pad 2: /Microphone/3.3V -> +3.3V
- J2 pad 1: Net-(J2-Pin_1) -> +BATT
- J3 pad 4: /Microphone/3.3V -> +3.3V
- J8 pad 2: /Microphone/3.3V -> +3.3V
- MK1 pad 5: /Microphone/3.3V -> +3.3V
- SW1 pad 2: /Microphone/3.3V -> +3.3V
- SW2 pad 2: /Microphone/3.3V -> +3.3V
- SW3 pad 2: /Microphone/3.3V -> +3.3V
- SW4 pad 2: /Microphone/3.3V -> +3.3V
- SW5 pad 2: /Microphone/3.3V -> +3.3V
- SW6 pad 2: /Microphone/3.3V -> +3.3V
- SW7 pad 2: /Microphone/3.3V -> +3.3V
- SW8 pad 2: /Microphone/3.3V -> +3.3V
- U10 pad 20: /Microphone/3.3V -> +3.3V
- U10 pad 21: /Microphone/3.3V -> +3.3V
- U2 pad 5: /Microphone/3.3V -> +3.3V
- U4 pad 100: /Microphone/3.3V -> +3.3V
- U4 pad 11: /Microphone/3.3V -> +3.3V
- U4 pad 27: /Microphone/3.3V -> +3.3V
- U4 pad 50: /Microphone/3.3V -> +3.3V
- U4 pad 6: Net-(BT1-+) -> +3.3V
- U4 pad 75: /Microphone/3.3V -> +3.3V
- U4 pad 8: OSC32_IN -> unconnected-(U4-PC14-Pad8)
- U4 pad 9: OSC32_OUT -> unconnected-(U4-PC15-Pad9)
- U5 pad 1: /Microphone/3.3V -> +3.3V
- U6 pad 5: /Microphone/3.3V -> +3.3V
- U6 pad 8: /Microphone/3.3V -> +3.3V
- U7 pad 14: Net-(BT2-+) -> +BATT
- U7 pad 2: /Microphone/3.3V -> +3.3V
- U8 pad 6: /Microphone/3.3V -> +3.3V
- U8 pad 8: /Microphone/3.3V -> +3.3V
Routing:
- net GND: track 0.00 -> 152.3 mm, vias 0 -> 38
- net +3.3V: track 0.00 -> 104.3 mm, vias 0 -> 13
- net +5V: track 0.00 -> 95.4 mm, vias 0 -> 7
- net +BATT: track 0.00 -> 74.7 mm, vias 0 -> 4
- net USB_PROT_D+: track 0.00 -> 45.1 mm, vias 0 -> 1
- net USB_PROT_D-: track 0.00 -> 44.4 mm, vias 0 -> 1
- net (no net): track 0.00 -> 43.7 mm
- net /Audio/1.8v: track 0.00 -> 36.5 mm
- net /OLED UI/Col3: track 0.00 -> 30.2 mm, vias 0 -> 2
- net /OLED UI/Col1: track 0.00 -> 28.1 mm, vias 0 -> 2
- net LIGHT_INT: track 0.00 -> 23.9 mm, vias 0 -> 1
- net /OLED UI/OLED_SCK: track 0.00 -> 18.6 mm, vias 0 -> 1
- net Net-(D8-K): track 0.00 -> 18.4 mm, vias 0 -> 2
- net /OLED UI/Col2: track 0.00 -> 18.4 mm
- net Net-(D9-K): track 0.00 -> 18.0 mm, vias 0 -> 2
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- added copper zone on In2.Cu, net +3.3V
- added copper zone on F.Cu, net GND
- added copper zone on In1.Cu, net GND
Other:
- copper layers 2 -> 4
