File: kicad/MP3player.kicad_pcb (KiCad board)
At the start: 6 copper layers, 50 x 70 mm, 148 parts, among them J1 USB_C_Receptacle_USB2.0_14P, J2 Conn_01x02, J3 Conn_01x05, J4 AudioJack3_Ground_SwitchTR, J5 Micro_SD_Card_Det2, J6 SMA, J7 SMA, J8 Conn_01x08, SW1 SW_Push, SW10 SW_Push, SW11 SW_Push, SW12 SW_Push, SW13 SW_Push, SW14 SW_Push, SW15 SW_Push, SW16 SW_Push, SW17 SW_Push, SW2 SW_Push, SW3 SW_Push, SW4 SW_Push, SW5 SW_Push, SW6 SW_Push, SW7 SW_Push, SW8 SW_Push, SW9 SW_Push, U1 USBLC6-2SC6, U10 Si4735-D60-GU, U11 BQ24090DGQ, U12 TPS613222ADBV, U2 TLV70233_SOT23-5, U3 TPS7A4701xRGW, U4 STM32H743VIT6, U5 ISL29035, U6 LSM6DSL, U7 DS3231M, U8 BME680, U9 CS43131-CNZR, Y1 8MHz TXC AA08000002

Commit message: fix images
Parts:
- added G***: LOGO, logo:linuxpenguin_cu, F.Cu at (65.0, 59.0)
- added G***: LOGO, logo:linuxpenguin-mask, F.Cu at (65.0, 59.0)
