File: kicad/MP3player.kicad_pcb (KiCad board)
At the start: 6 copper layers, 50 x 70 mm, 150 parts, among them J1 USB_C_Receptacle_USB2.0_14P, J2 Conn_01x02, J3 Conn_01x05, J4 AudioJack3_Ground_SwitchTR, J5 Micro_SD_Card_Det2, J6 SMA, J7 SMA, J8 Conn_01x08, SW1 SW_Push, SW10 SW_Push, SW11 SW_Push, SW12 SW_Push, SW13 SW_Push, SW14 SW_Push, SW15 SW_Push, SW16 SW_Push, SW17 SW_Push, SW2 SW_Push, SW3 SW_Push, SW4 SW_Push, SW5 SW_Push, SW6 SW_Push, SW7 SW_Push, SW8 SW_Push, SW9 SW_Push, U1 USBLC6-2SC6, U10 Si4735-D60-GU, U11 BQ24090DGQ, U12 TPS613222ADBV, U2 TLV70233_SOT23-5, U3 TPS7A4701xRGW, U4 STM32H743VIT6, U5 ISL29035, U6 LSM6DSL, U7 DS3231M, U8 BME680, U9 CS43131-CNZR, Y1 8MHz TXC AA08000002

Commit message: a
Parts:
- L1: footprint Inductor_SMD:L_0805_2012Metric -> Inductor_SMD:L_1206_3216Metric
- moved L1 0.50 mm to (44.0, 58.0)
Changed lines of the file:
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@@
 		)
 	)
-	(footprint "Inductor_SMD:L_0805_2012Metric"
+	(footprint "Inductor_SMD:L_1206_3216Metric"
 		(layer "F.Cu")
-		(at 44.5 58)
-		(descr "Inductor SMD 0805 (2012 Metric), square (rectangular) end terminal, IPC-7351 nominal, (Body size source: IPC-SM-782 page 80, https://www.pcb-3d.com/wordpress/wp-content/uploads/ipc-sm-782a_amendment_1_and_2.pdf)")
+		(at 44 58)
+		(descr "Inductor SMD 1206 (3216 Metric), square (rectangular) end terminal, IPC-7351 nominal, (Body size source: IPC-SM-782 page 80, https://www.pcb-3d.com/wordpress/wp-content/uploads/ipc-sm-782a_amendment_1_and_2.pdf)")
 		(tags "inductor")
 		(property "Reference" "L1"
-			(at -3 0 0)
+			(at -3.5 -0.5 0)
 			(layer "F.SilkS")
 			(effects
@@
 		)
 		(property "Value" "450uH"
-			(at 0 1.55 0)
+			(at 0 1.9 0)
 			(layer "F.Fab")
 			(effects
@@
 		(duplicate_pad_numbers_are_jumpers no)
 		(fp_line
-			(start -0.399622 -0.56)
-			(end 0.399622 -0.56)
+			(start -0.835242 -0.91)
+			(end 0.835242 -0.91)
 			(stroke
 				(width 0.12)
@@
 		)
 		(fp_line
-			(start -0.399622 0.56)
-			(end 0.399622 0.56)
+			(start -0.835242 0.91)
+			(end 0.835242 0.91)
 			(stroke
 				(width 0.12)
@@
 		)
 		(fp_rect
-			(start -1.75 -0.85)
-			(end 1.75 0.85)
+			(start -2.35 -1.2)
+			(end 2.35 1.2)
 			(stroke
 				(width 0.05)
@@
 		)
 		(fp_rect
-			(start -1 -0.45)
-			(end 1 0.45)
+			(start -1.6 -0.8)
+			(end 1.6 0.8)
 			(stroke
 				(width 0.1)
@@
 			(effects
 				(font
-					(size 0.5 0.5)
-					(thickness 0.08)
+					(size 0.8 0.8)
+					(thickness 0.12)
 				)
 			)
 		)
 		(pad "1" smd roundrect
-			(at -1.0625 0)
-			(size 0.875 1.2)
+			(at -1.575 0)
+			(size 1.05 1.9)
 			(layers "F.Cu" "F.Mask" "F.Paste")
-			(roundrect_rratio 0.25)
+			(roundrect_rratio 0.238095)
 			(net "Net-(J7-In)")
 			(pinfunction "1_1")
@@
 		)
 		(pad "2" smd roundrect
-			(at 1.0625 0)
-			(size 0.875 1.2)
+			(at 1.575 0)
+			(size 1.05 1.9)
 			(layers "F.Cu" "F.Mask" "F.Paste")
-			(roundrect_rratio 0.25)
+			(roundrect_rratio 0.238095)
 			(net "GND")
 			(pinfunction "2_2")
@@
 		)
 		(embedded_fonts no)
-		(model "${KICAD10_3DMODEL_DIR}/Inductor_SMD.3dshapes/L_0805_2012Metric.step"
+		(model "${KICAD10_3DMODEL_DIR}/Inductor_SMD.3dshapes/L_1206_3216Metric.step"
 			(offset
 				(xyz 0 0 0)
@@
 	)
 	(segment
-		(start 43.4375 58)
+		(start 43.4375 55.7875)
+		(end 43.725 55.5)
+		(width 0.2)
+		(layer "F.Cu")
+		(net "Net-(J7-In)")
+	)
+	(segment
+		(start 43.4375 56.9875)
 		(end 43.4375 55.7875)
 		(width 0.2)
@@
 	)
 	(segment
-		(start 43.4375 55.7875)
-		(end 43.725 55.5)
+		(start 42.425 58)
+		(end 43.4375 56.9875)
 		(width 0.2)
 		(layer "F.Cu")
