File: kicad/microphone.kicad_sch (KiCad schematic)
At the start: 3 parts

Commit message: almost done!
Parts:
- C129: footprint (none) -> Capacitor_SMD:C_0603_1608Metric
Changed lines of the file:
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@@
 			)
 		)
-		(property "Footprint" ""
+		(property "Footprint" "Capacitor_SMD:C_0603_1608Metric"
 			(at 41.91 22.86 0)
 			(hide yes)

Commit message: general changes
Parts:
- R20: footprint (none) -> Resistor_SMD:R_0603_1608Metric
- renumbered C129 to C53
Changed lines of the file:
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@@
 		(dnp no)
 		(fields_autoplaced yes)
-		(property "Reference" "C129"
+		(property "Reference" "C53"
 			(at 44.45 21.5962 0)
 			(show_name no)
@@
 			(project "MP3player"
 				(path "/c86fdb70-ebb0-4c87-946f-42a0fbefb388/3c7a344c-7f88-4b5c-bff2-9cbba23de578"
-					(reference "C129")
+					(reference "C53")
 					(unit 1)
 				)
@@
 			)
 		)
-		(property "Footprint" ""
+		(property "Footprint" "Resistor_SMD:R_0603_1608Metric"
 			(at 34.29 39.37 0)
 			(hide yes)
