File: kicad/oledui.kicad_sch (KiCad schematic)
At the start: 0 parts

Commit message: almost done schematic
Parts:
- added D1, D2, D3: ACDSV6-4448TI-G, Package_TO_SOT_SMD:SOT-23-3, symbol Diode:ACDSV6-4448TI-G
- added J7: Conn_01x08, Connector_PinHeader_2.54mm:PinHeader_1x08_P2.54mm_Vertical, symbol Connector_Generic:Conn_01x08
- added R12, R13, R14, R15, R16, R17, R18, R19: 10k, symbol Device:R_Small_US
- added SW1, SW11, SW2, SW3, SW4, SW5, SW6, SW7: SW_Push, Button_Switch_SMD:Panasonic_EVQPUM_EVQPUD, symbol Switch:SW_Push
- added SW10, SW12, SW13, SW14, SW15, SW16, SW17, SW8, SW9: SW_Push, Button_Switch_THT:Push_E-Switch_KS01Q01, symbol Switch:SW_Push
Connections:
- net BTN_POWER: now also R12.2, SW1.1
- net BTN_VOL_DOWN: now also R14.2, SW3.1
- net BTN_VOL_UP: now also R13.2, SW2.1
- net OLED_CS: now also J7.7 (Pin_7)
- net OLED_DC: now also J7.6 (Pin_6)
- net OLED_MOSI: now also J7.4 (Pin_4)
- net OLED_RST: now also J7.5 (Pin_5)
- net OLED_SCK: now also J7.3 (Pin_3)
- new net: D3.1 (A), SW15.2
- new net: D1.1 (A), SW8.2
- new net: D3.2 (A), SW16.2
- new net: D1.3 (A), SW10.2
- new net: D3.3 (A), SW17.2
- new net: D2.2 (A), SW13.2
- new net: D2.3 (A), SW14.2
- new net: D2.1 (A), SW12.2
- new net: D1.2 (A), SW9.2
- new net 3.3v: J7.2 (Pin_2), SW1.2, SW11.2, SW2.2, SW3.2, SW4.2, SW5.2, SW6.2, SW7.2
- new net BTN_BOOT0: R19.2, SW11.1
- new net BTN_LOCK: R15.2, SW4.1
- new net BTN_RECORD: R16.2, SW5.1
- new net BTN_RST: R18.2, SW7.1
- new net BTN_USER: R17.2, SW6.1
- new net Col1: D1.4 (K), D1.5 (K), D1.6 (K)
- new net Col2: D2.4 (K), D2.5 (K), D2.6 (K)
- new net Col3: D3.4 (K), D3.5 (K), D3.6 (K)
- new net GND: J7.1 (Pin_1), R12.1, R13.1, R14.1, R15.1, R16.1, R17.1, R18.1, R19.1
- new net OLED_BL: J7.8 (Pin_8)
- new net Row1: SW12.1, SW15.1, SW8.1
- new net Row2: SW13.1, SW16.1, SW9.1
- new net Row3: SW10.1, SW14.1, SW17.1
Other:
- note added: "Boot"
- note added: "BottomLeft"
- note added: "Left"
- note added: "Lock"
- note added: "Power switch"
- note added: "Record"
- note added: "Reset"
- note added: "SWITCH TO MATRIX NEXT REVISION"
- note added: "Top"
- note added: "TopLeft"
- note added: "User programmable buton"
- note added: "Volume UP"
- note added: "Volume down"

Commit message: almost done!
Parts:
- removed SW9: SW_Push, Button_Switch_THT:Push_E-Switch_KS01Q01, symbol Switch:SW_Push
- added SW11: SW_Push, Button_Switch_SMD:SW_Push_1P1T_NO_CK_KSC9xxJ, symbol Switch:SW_Push
- SW10, SW12, SW13, SW14, SW15, SW16, SW17: footprint Button_Switch_THT:Push_E-Switch_KS01Q01 -> Button_Switch_SMD:SW_Push_1P1T_NO_CK_KSC9xxJ
- SW9: renamed from SW8; footprint Button_Switch_THT:Push_E-Switch_KS01Q01 -> Button_Switch_SMD:SW_Push_1P1T_NO_CK_KSC9xxJ
- renumbered J7 to J8, R18 to R12, R19 to R13, R12 to R14, R13 to R15, R14 to R16, R15 to R17, R16 to R18, R17 to R19, SW7 to SW1, SW11 to SW2, SW1 to SW3, SW2 to SW4, SW3 to SW5, SW4 to SW6, SW5 to SW7, SW6 to SW8
Connections:
- net Row2: now also SW10.1
- net Row3: now also SW11.1; no longer SW10.1
- net at D1.3 (A): now also SW11.2; no longer SW10.2
- net at D1.2 (A): now also SW10.2

Commit message: general changes
Parts:
- D1, D2, D3: footprint Package_TO_SOT_SMD:SOT-23-3 -> Package_TO_SOT_SMD:SOT-363_SC-70-6
- J8: footprint Connector_PinHeader_2.54mm:PinHeader_1x08_P2.54mm_Vertical -> Connector_PinHeader_2.54mm:PinHeader_1x08_P2.54mm_Vertical_SMD_Pin1Right
- R12, R13, R14, R15, R16, R17, R18, R19: footprint (none) -> Resistor_SMD:R_0603_1608Metric
- SW10, SW11, SW12, SW13, SW14, SW15, SW16, SW17, SW9: footprint Button_Switch_SMD:SW_Push_1P1T_NO_CK_KSC9xxJ -> Button_Switch_SMD:SW_Push_1P1T_NO_CK_KMR2
