File: kicad/power.kicad_sch (KiCad schematic)
At the start: 17 parts, among them J1 USB_C_Receptacle_USB2.0_14P, U1 USBLC6-2SC6, U2 TLV70233_SOT23-5, U3 TPS7A4701xRGW

Commit message: almost done!
Parts:
- removed BT1: 18650, Battery:BatteryHolder_Keystone_1042_1x18650, symbol Device:Battery_Cell
- added J2: Conn_01x02, Connector_JST:JST_PH_B2B-PH-K_1x02_P2.00mm_Vertical, symbol Connector_Generic:Conn_01x02
- C1, C2, C3, C4, C5, C6, C7: footprint (none) -> Capacitor_SMD:C_0603_1608Metric
- J1: footprint (none) -> Connector_USB:USB_C_Receptacle_HRO_TYPE-C-31-M-12
Connections:
- net GND: now also J2.2 (Pin_2)
- net at A1.3 (VBAT+), A1.4 (VBAT+): now also J2.1 (Pin_1)
Changed lines of the file:
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@@
 	(wire
 		(pts
-			(xy 38.1 105.41) (xy 38.1 106.68)
-		)
-		(stroke
-			(width 0)
-			(type default)
-		)
-	)
-	(wire
-		(pts
-			(xy 38.1 86.36) (xy 38.1 97.79)
+			(xy 38.1 102.87) (xy 38.1 106.68)
+		)
+		(stroke
+			(width 0)
+			(type default)
+		)
+	)
+	(wire
+		(pts
+			(xy 38.1 86.36) (xy 38.1 100.33)
 		)
 		(stroke
@@
 			)
 		)
-		(property "Footprint" ""
+		(property "Footprint" "Capacitor_SMD:C_0603_1608Metric"
 			(at 227.33 35.56 0)
 			(hide yes)
@@
 			)
 		)
-		(property "Footprint" ""
+		(property "Footprint" "Capacitor_SMD:C_0603_1608Metric"
 			(at 270.51 35.56 0)
 			(hide yes)
@@
 	)
 	(symbol
+		(lib_id "Connector_Generic:Conn_01x02")
+		(at 43.18 100.33 0)
+		(unit 1)
+		(body_style 1)
+		(exclude_from_sim no)
+		(in_bom yes)
+		(on_board yes)
+		(in_pos_files yes)
+		(dnp no)
+		(fields_autoplaced yes)
+		(property "Reference" "J2"
+			(at 45.72 100.3299 0)
+			(show_name no)
+			(do_not_autoplace no)
+			(effects
+				(font
+					(size 1.27 1.27)
+				)
+				(justify left)
+			)
+		)
+		(property "Value" "Conn_01x02"
+			(at 45.72 102.8699 0)
+			(show_name no)
+			(do_not_autoplace no)
+			(effects
+				(font
+					(size 1.27 1.27)
+				)
+				(justify left)
+			)
+		)
+		(property "Footprint" "Connector_JST:JST_PH_B2B-PH-K_1x02_P2.00mm_Vertical"
+			(at 43.18 100.33 0)
+			(hide yes)
+			(show_name no)
+			(do_not_autoplace no)
+			(effects
+				(font
+					(size 1.27 1.27)
+				)
+			)
+		)
+		(property "Datasheet" ""
+			(at 43.18 100.33 0)
+			(hide yes)
+			(show_name no)
+			(do_not_autoplace no)
+			(effects
+				(font
+					(size 1.27 1.27)
+				)
+			)
+		)
+		(property "Description" "Generic connector, single row, 01x02, script generated (kicad-library-utils/schlib/autogen/connector/)"
+			(at 43.18 100.33 0)
+			(hide yes)
+			(show_name no)
+			(do_not_autoplace no)
+			(effects
+				(font
+					(size 1.27 1.27)
+				)
+			)
+		)
+		(pin "1"
+		)
+		(pin "2"
+		)
+		(instances
+			(project "MP3player"
+				(path "/c86fdb70-ebb0-4c87-946f-42a0fbefb388/44773f7f-d06f-4f25-afe6-dcac6b52c94d"
+					(reference "J2")
+					(unit 1)
+				)
+			)
+		)
+	)
+	(symbol
 		(lib_id "Device:C_Small")
 		(at 163.83 55.88 0)
@@
 			)
 		)
-		(property "Footprint" ""
+		(property "Footprint" "Capacitor_SMD:C_0603_1608Metric"
 			(at 163.83 55.88 0)
 			(hide yes)
@@
 			)
 		)
-		(property "Footprint" ""
+		(property "Footprint" "Connector_USB:USB_C_Receptacle_HRO_TYPE-C-31-M-12"
 			(at 39.37 41.91 0)
 			(hide yes)
@@
 			)
 		)
-		(property "Footprint" ""
+		(property "Footprint" "Capacitor_SMD:C_0603_1608Metric"
 			(at 173.99 55.88 0)
 			(hide yes)
@@
 			)
 		)
-		(property "Footprint" ""
+		(property "Footprint" "Capacitor_SMD:C_0603_1608Metric"
 			(at 200.66 55.88 0)
 			(hide yes)
@@
 	)
 	(symbol
-		(lib_id "Device:Battery_Cell")
-		(at 38.1 102.87 0)
-		(unit 1)
-		(body_style 1)
-		(exclude_from_sim no)
-		(in_bom yes)
-		(on_board yes)
-		(in_pos_files yes)
-		(dnp no)
-		(fields_autoplaced yes)
-		(property "Reference" "BT1"
-			(at 41.91 99.7584 0)
-			(show_name no)
-			(do_not_autoplace no)
-			(effects
-				(font
-					(size 1.27 1.27)
-				)
-				(justify left)
-			)
-		)
-		(property "Value" "18650"
-			(at 41.91 102.2984 0)
-			(show_name no)
-			(do_not_autoplace no)
-			(effects
-				(font
-					(size 1.27 1.27)
-				)
-				(justify left)
-			)
-		)
-		(property "Footprint" "Battery:BatteryHolder_Keystone_1042_1x18650"
-			(at 38.1 101.346 90)
-			(hide yes)
-			(show_name no)
-			(do_not_autoplace no)
-			(effects
-				(font
-					(size 1.27 1.27)
-				)
-			)
-		)
-		(property "Datasheet" ""
-			(at 38.1 101.346 90)
-			(hide yes)
-			(show_name no)
-			(do_not_autoplace no)
-			(effects
-				(font
-					(size 1.27 1.27)
-				)
-			)
-		)
-		(property "Description" "Single-cell battery"
-			(at 38.1 102.87 0)
-			(hide yes)
-			(show_name no)
-			(do_not_autoplace no)
-			(effects
-				(font
-					(size 1.27 1.27)
-				)
-			)
-		)
-		(property "Sim.Device" "V"
-			(at 38.1 102.87 0)
-			(hide yes)
-			(show_name no)
-			(do_not_autoplace no)
-			(effects
-				(font
-					(size 1.27 1.27)
-				)
-			)
-		)
-		(property "Sim.Type" "DC"
-			(at 38.1 102.87 0)
-			(hide yes)
-			(show_name no)
-			(do_not_autoplace no)
-			(effects
-				(font
-					(size 1.27 1.27)
-				)
-			)
-		)
-		(property "Sim.Pins" "1=+ 2=-"
-			(at 38.1 102.87 0)
-			(hide yes)
-			(show_name no)
-			(do_not_autoplace no)
-			(effects
-				(font
-					(size 1.27 1.27)
-				)
-			)
-		)
-		(pin "1"
-		)
-		(pin "2"
-		)
-		(instances
-			(project "MP3player"
-				(path "/c86fdb70-ebb0-4c87-946f-42a0fbefb388/44773f7f-d06f-4f25-afe6-dcac6b52c94d"
-					(reference "BT1")
-					(unit 1)
-				)
-			)
-		)
-	)
-	(symbol
 		(lib_id "PMM:PMM")
 		(at 88.9 101.6 0)
@@
 			)
 		)
-		(property "Footprint" ""
+		(property "Footprint" "Capacitor_SMD:C_0603_1608Metric"
 			(at 261.62 59.69 0)
 			(hide yes)
@@
 			)
 		)
-		(property "Footprint" ""
+		(property "Footprint" "Capacitor_SMD:C_0603_1608Metric"
 			(at 210.82 55.88 0)
 			(hide yes)

Commit message: general changes
Parts:
- removed A1: PMM, PMM:PMM, symbol PMM:PMM
- added C59: 1uF, Capacitor_SMD:C_0603_1608Metric, symbol Device:C_Small
- added C60: 4.7uF, Capacitor_SMD:C_0603_1608Metric, symbol Device:C_Small
- added C61: 22uF, Capacitor_SMD:C_0603_1608Metric, symbol Device:C_Small
- added C62: 120pF, Capacitor_SMD:C_0603_1608Metric, symbol Device:C_Small
- added D10: BAT54W, Package_TO_SOT_SMD:SOT-323_SC-70, symbol Diode:BAT54W
- added D8, D9: LED, LED_SMD:LED_0603_1608Metric, symbol Device:LED
- added L2: 2.2uH, Inductor_SMD:L_0805_2012Metric, symbol Device:L
- added R21, R22: 1.5k, Resistor_SMD:R_0603_1608Metric, symbol Device:R_Small_US
- added R23, R25: 1.1k, Resistor_SMD:R_0603_1608Metric, symbol Device:R_Small_US
- added R24: 11k, Resistor_SMD:R_0603_1608Metric, symbol Device:R_Small_US
- added R26: 5.11R, Resistor_SMD:R_0603_1608Metric, symbol Device:R_Small_US
- added TH1: 10k, Resistor_SMD:R_0603_1608Metric, symbol Device:Thermistor_NTC_US
- added U11: BQ24090DGQ, Package_SO:HVSSOP-10-1EP_3x3mm_P0.5mm_EP1.83x1.89mm, symbol Battery_Management:BQ24090DGQ
- added U12: TPS613222ADBV, Package_TO_SOT_SMD:SOT-23-5, symbol Regulator_Switching:TPS613222ADBV
- R1, R2, R3, R4: footprint (none) -> Resistor_SMD:R_0603_1608Metric
Connections:
- net +5V: now also C61.1, C62.2, D10.3 (K), U12.4 (VOUT)
- net GND: now also C59.2, C60.2, C61.2, R23.2, R24.2, R25.2, TH1.2, U11.11 (VSS), U11.3 (VSS), U12.2 (GND)
- net VBUS: now also C59.1, U11.1 (IN)
- net +BATT: now reaches J2.1 (Pin_1)
- net +BATT: now also C60.1, L2.1, R21.1, R22.1, U11.10 (OUT)
- new net: R23.1, U11.4 (PRETERM)
- new net: R24.1, U11.7 (ISET2)
- new net: R25.1, U11.2 (ISET)
- new net: D10.1 (A), L2.2, R26.1, U12.1 (SW)
- new net: C62.1, R26.2
- new net: D9.2 (A), R22.2
- new net: D8.2 (A), R21.2
- new net: D9.1 (K), U11.5 (~{PG})
- new net: D8.1 (K), U11.8 (~{CHG})
- new net: TH1.1, U11.9 (TS)
- no-connect marks 23 -> 5
