File: kicad/stm32core.kicad_sch (KiCad schematic)
At the start: 32 parts, among them J2 Conn_01x05, U7 STM32H743VIT6, U8 DS3231M, Y1 8MHz, Y2 32.768KHz

Commit message: almost done schematic
Parts:
- added C16, C27, C28, C29, C31, C33: 100nF, symbol Device:C_Small
- added U5: ISL29035, OptoDevice:Renesas_DFN-6_1.5x1.6mm_P0.5mm, symbol Sensor_Optical:ISL29035
- added U6: LSM6DSL, Package_LGA:LGA-14_3x2.5mm_P0.5mm_LayoutBorder3x4y, symbol Sensor_Motion:LSM6DSL
- added U8: BME680, Package_LGA:Bosch_LGA-8_3x3mm_P0.8mm_ClockwisePinNumbering, symbol Sensor:BME680
- renumbered BT3 to BT2, BT4 to BT3, C27 to C10, C28 to C11, C29 to C12, C30 to C13, C31 to C14, C32 to C15, C33 to C17, C34 to C18, C35 to C19, C36 to C20, C37 to C21, C38 to C22, C39 to C23, C40 to C24, C41 to C25, C42 to C26, C43 to C30, C44 to C32, C25 to C8, C26 to C9, R22 to R5, R23 to R6, R24 to R7, R25 to R8, U7 to U4, U8 to U7
Connections:
- net BTN_BACK is gone; now on net BTN_POWER: U4.22 (PA0)
- net BTN_MENU is gone; now on net BTN_VOL_UP: U4.23 (PA1)
- net BTN_PREV is gone; now on net BTN_VOL_DOWN: U4.24 (PA2)
- net OLED_MISO is gone; now on net OLED_RST: U4.30 (PA6)
- net VREF is gone; now on net CLEANFILTERED3V3: U4.20 (VREF+)
- net 3.3V: now also C27.1, C28.1, C29.1, C31.1, C33.1, U5.1 (VDD), U6.5 (VDDIO), U6.8 (VDD), U8.6 (VDDIO), U8.8 (VDD)
- net BTN_POWER: no longer U4.18 (PC3_C)
- net BTN_VOL_DOWN: no longer U4.16 (PC1)
- net BTN_VOL_UP: no longer U4.17 (PC2_C)
- net GND: now also C16.2, C27.2, C28.2, C29.2, C31.2, C33.2, U5.2 (GND), U6.6 (GND), U6.7 (GND), U8.1 (GND), U8.7 (GND)
- net LED_MOSI: now also U4.52 (PB13); no longer U4.54 (PB15)
- net LED_SCK: now also U4.47 (PB11); no longer U4.52 (PB13)
- net OLED_RST: no longer U4.15 (PC0)
- net SDMMC_CMD: now also U4.7 (PC13); no longer U4.83 (PD2)
- net CLEANFILTERED3V3: now reaches C22.1, C23.1, C24.1, FB1.1, U4.21 (VDDA)
- net CLEANFILTERED3V3: now also C16.1
- net I2S_MCLK: now reaches U4.1 (PE2)
- net Col1: now reaches U4.34 (PB0)
- net Col2: now reaches U4.35 (PB1)
- net Col3: now reaches U4.36 (PB2)
- net SENSORS_SPI1_MOSI: now reaches U4.37 (PE7)
- net SENSORS_SPI1_MOSI: now also U8.3 (SDI)
- net I2S_LRCLK: now reaches U4.41 (PE11)
- net I2S_BCLK: now reaches U4.42 (PE12)
- net SENSORS_SPI1_SCK: now reaches U4.43 (PE13)
- net SENSORS_SPI1_SCK: now also U8.4 (SCK)
- net I2S_SDOUT: now reaches U4.44 (PE14)
- net RADIO_I2S_BCLK: now reaches U4.46 (PB10)
- net SENSORS_SPI1_MISO: now reaches U4.5 (PE6)
- net SENSORS_SPI1_MISO: now also U8.5 (SDO)
- net RADIO_I2S_LRCLK: now reaches U4.51 (PB12)
- net RADIO_GP1: now reaches U4.53 (PB14)
- net PMM_TX: now reaches U4.55 (PD8)
- net PMM_RX: now reaches U4.56 (PD9)
- net PMM_SHDN: now reaches U4.57 (PD10)
- net RADIO_RST: now reaches U4.61 (PD14)
- net PMM_INIT: now reaches U4.62 (PD15)
- net SDMMC_DET: now reaches U4.64 (PC7)
- net MIC_CHANNEL: now reaches U4.77 (PA15)
- net AUDIO_INT: now reaches U4.84 (PD3)
- net AUDIO_RESET: now reaches U4.85 (PD4)
- net PMM_FORCE: now reaches U4.88 (PD7)
- net Row1: now reaches U4.89 (PB3)
- net Row2: now reaches U4.90 (PB4)
- net AUDIO_SDA: now reaches U4.97 (PE0)
- net AUDIO_SCL: now reaches U4.98 (PE1)
- net BTN_NEXT renamed BTN_LOCK
- net BTN_PLAY renamed BTN_RECORD
- net MAX17263_INT renamed OLED_BL
- new net BTN_USER: U4.16 (PC1)
- new net GAS_CS: U8.2 (CSB)
- new net IMU_INT1: U6.4 (INT1)
- new net IMU_INT2: U6.9 (INT2)
- new net LIGHT_INT: U5.4 (~INT)
- new net RADIO_I2S_DATA: U4.54 (PB15)
- new net Row3: U4.15 (PC0)
- new net SENSORS_I2C_SCL: U5.5 (SCL)
- new net SENSORS_I2C_SDA: U5.6 (SDA)
- no-connect marks 0 -> 1
Other:
- note added: "Light Sensor"
- note added: "imu"
- note added: "temp pres humi gas"
- moved on the sheet: R6

Commit message: add sensors
Connections:
- net GAS_CS: now also U4.40 (PE10)
- net IMU_CS: now also U4.38 (PE8), U6.12 (CS)
- net IMU_INT1: now also U4.39 (PE9)
- net IMU_INT2: now also U4.17 (PC2_C)
- net LIGHT_INT: now also U4.18 (PC3_C)
- net SENSORS_I2C_SCL: now also U4.81 (PD0)
- net SENSORS_I2C_SDA: now also U4.82 (PD1)
- net SENSORS_SPI1_MISO: now also U4.86 (PD5), U6.1 (SDO/SA0)
- net SENSORS_SPI1_MOSI: now also U4.87 (PD6), U6.14 (SDA)
- net SENSORS_SPI1_SCK: now also U6.13 (SCL)
- no-connect marks 1 -> 8

Commit message: almost done!
Parts:
- C10, C11, C12, C13, C14, C15, C16, C17, C18, C19, C20, C21, C22, C23, C24, C25, C26, C27, C28, C29, C30, C31, C32, C33, C8, C9: footprint (none) -> Capacitor_SMD:C_0603_1608Metric
- FB1: footprint (none) -> Inductor_SMD:L_0603_1608Metric
- J3: renamed from J2; footprint (none) -> Connector_PinHeader_2.54mm:PinHeader_1x05_P2.54mm_Vertical
- renumbered BT2 to BT1, BT3 to BT2
Changed lines of the file:
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@@
 			)
 		)
-		(property "Footprint" ""
+		(property "Footprint" "Capacitor_SMD:C_0603_1608Metric"
 			(at 156.21 31.75 0)
 			(hide yes)
@@
 		(dnp no)
 		(fields_autoplaced yes)
-		(property "Reference" "BT2"
+		(property "Reference" "BT1"
 			(at 87.63 33.7184 0)
 			(show_name no)
@@
 			(project "MP3player"
 				(path "/c86fdb70-ebb0-4c87-946f-42a0fbefb388/6908e98e-7fb1-4e28-9490-dbce6fc1994c"
-					(reference "BT2")
+					(reference "BT1")
 					(unit 1)
 				)
@@
 		(dnp no)
 		(fields_autoplaced yes)
-		(property "Reference" "BT3"
+		(property "Reference" "BT2"
 			(at 257.81 22.2884 0)
 			(show_name no)
@@
 			(project "MP3player"
 				(path "/c86fdb70-ebb0-4c87-946f-42a0fbefb388/6908e98e-7fb1-4e28-9490-dbce6fc1994c"
-					(reference "BT3")
+					(reference "BT2")
 					(unit 1)
 				)
@@
 			)
 		)
-		(property "Footprint" ""
+		(property "Footprint" "Capacitor_SMD:C_0603_1608Metric"
 			(at 114.3 31.75 0)
 			(hide yes)
@@
 			)
 		)
-		(property "Footprint" ""
+		(property "Footprint" "Capacitor_SMD:C_0603_1608Metric"
 			(at 64.77 167.64 0)
 			(hide yes)
@@
 			)
 		)
-		(property "Footprint" ""
+		(property "Footprint" "Capacitor_SMD:C_0603_1608Metric"
 			(at 33.02 157.48 0)
 			(hide yes)
@@
 			)
 		)
-		(property "Footprint" ""
+		(property "Footprint" "Capacitor_SMD:C_0603_1608Metric"
 			(at 124.46 31.75 0)
 			(hide yes)
@@
 			)
 		)
-		(property "Footprint" ""
+		(property "Footprint" "Capacitor_SMD:C_0603_1608Metric"
 			(at 63.5 25.4 0)
 			(hide yes)
@@
 			)
 		)
-		(property "Footprint" ""
+		(property "Footprint" "Capacitor_SMD:C_0603_1608Metric"
 			(at 147.32 31.75 0)
 			(hide yes)
@@
 			)
 		)
-		(property "Footprint" ""
+		(property "Footprint" "Capacitor_SMD:C_0603_1608Metric"
 			(at 35.56 53.34 0)
 			(hide yes)
@@
 			)
 		)
-		(property "Footprint" ""
+		(property "Footprint" "Inductor_SMD:L_0603_1608Metric"
 			(at 142.24 27.178 90)
 			(hide yes)
@@
 			)
 		)
-		(property "Footprint" ""
+		(property "Footprint" "Capacitor_SMD:C_0603_1608Metric"
 			(at 240.03 22.86 0)
 			(hide yes)
@@
 			)
 		)
-		(property "Footprint" ""
+		(property "Footprint" "Capacitor_SMD:C_0603_1608Metric"
 			(at 57.15 63.5 0)
 			(hide yes)
@@
 			)
 		)
-		(property "Footprint" ""
+		(property "Footprint" "Capacitor_SMD:C_0603_1608Metric"
 			(at 33.02 25.4 0)
 			(hide yes)
@@
 			)
 		)
-		(property "Footprint" ""
+		(property "Footprint" "Capacitor_SMD:C_0603_1608Metric"
 			(at 43.18 25.4 0)
 			(hide yes)
@@
 			)
 		)
-		(property "Footprint" ""
+		(property "Footprint" "Capacitor_SMD:C_0603_1608Metric"
 			(at 17.78 157.48 0)
 			(hide yes)
@@
 			)
 		)
-		(property "Footprint" ""
+		(property "Footprint" "Capacitor_SMD:C_0603_1608Metric"
 			(at 229.87 118.11 0)
 			(hide yes)
@@
 			)
 		)
-		(property "Footprint" ""
+		(property "Footprint" "Capacitor_SMD:C_0603_1608Metric"
 			(at 17.78 184.15 0)
 			(hide yes)
@@
 			)
 		)
-		(property "Footprint" ""
+		(property "Footprint" "Capacitor_SMD:C_0603_1608Metric"
 			(at 33.02 184.15 0)
 			(hide yes)
@@
 			)
 		)
-		(property "Footprint" ""
+		(property "Footprint" "Capacitor_SMD:C_0603_1608Metric"
 			(at 73.66 25.4 0)
 			(hide yes)
@@
 			)
 		)
-		(property "Footprint" ""
+		(property "Footprint" "Capacitor_SMD:C_0603_1608Metric"
 			(at 186.69 68.58 0)
 			(hide yes)
@@
 			)
 		)
-		(property "Footprint" ""
+		(property "Footprint" "Capacitor_SMD:C_0603_1608Metric"
 			(at 222.25 24.13 0)
 			(hide yes)
@@
 			)
 		)
-		(property "Footprint" ""
+		(property "Footprint" "Capacitor_SMD:C_0603_1608Metric"
 			(at 74.93 167.64 0)
 			(hide yes)
@@
 			)
 		)
-		(property "Footprint" ""
+		(property "Footprint" "Capacitor_SMD:C_0603_1608Metric"
 			(at 72.39 35.56 0)
 			(hide yes)
@@
 			)
 		)
-		(property "Footprint" ""
+		(property "Footprint" "Capacitor_SMD:C_0603_1608Metric"
 			(at 200.66 68.58 0)
 			(hide yes)
@@
 			)
 		)
-		(property "Footprint" ""
+		(property "Footprint" "Capacitor_SMD:C_0603_1608Metric"
 			(at 162.56 138.43 0)
 			(hide yes)
@@
 			)
 		)
-		(property "Footprint" ""
+		(property "Footprint" "Capacitor_SMD:C_0603_1608Metric"
 			(at 250.19 118.11 0)
 			(hide yes)
@@
 			)
 		)
-		(property "Footprint" ""
+		(property "Footprint" "Capacitor_SMD:C_0603_1608Metric"
 			(at 135.89 31.75 0)
 			(hide yes)
@@
 			)
 		)
-		(property "Footprint" ""
+		(property "Footprint" "Capacitor_SMD:C_0603_1608Metric"
 			(at 53.34 25.4 0)
 			(hide yes)
@@
 		(dnp no)
 		(fields_autoplaced yes)
-		(property "Reference" "J2"
+		(property "Reference" "J3"
 			(at 185.42 33.0199 0)
 			(show_name no)
@@
 			)
 		)
-		(property "Footprint" ""
+		(property "Footprint" "Connector_PinHeader_2.54mm:PinHeader_1x05_P2.54mm_Vertical"
 			(at 182.88 34.29 0)
 			(hide yes)
@@
 			(project "MP3player"
 				(path "/c86fdb70-ebb0-4c87-946f-42a0fbefb388/6908e98e-7fb1-4e28-9490-dbce6fc1994c"
-					(reference "J2")
+					(reference "J3")
 					(unit 1)
 				)

Commit message: general changes
Parts:
- removed BT1: CR2032, Battery:BatteryHolder_Keystone_3002_1x2032, symbol Device:Battery_Cell
- removed BT2: Battery_Cell, Battery:BatteryHolder_Keystone_3002_1x2032, symbol Device:Battery_Cell
- removed C12, C9: 8pF, Capacitor_SMD:C_0603_1608Metric, symbol Device:C_Small
- removed Y2: 32.768KHz, symbol Device:Crystal
- C11, C8: value 18pF -> 12pF
- R5, R6, R7, R8: footprint (none) -> Resistor_SMD:R_0603_1608Metric
- Y1: value 8MHz -> 8MHz TXC AA08000002; footprint (none) -> Crystal:Crystal_SMD_5032-2Pin_5.0x3.2mm
Connections:
- net 3.3V: now also C19.1, U4.6 (VBAT)
- net GND: now also C10.2, C14.2, C15.2, C17.2, C20.2
- net +BATT: now reaches C32.1, U7.14 (VBAT)
- net OSC32_IN: no longer names the net of U4.8 (PC14)
- net OSC32_OUT: no longer names the net of U4.9 (PC15)
- net PMM_FORCE: no longer names the net of U4.88 (PD7)
- net PMM_INIT: no longer names the net of U4.62 (PD15)
- net PMM_RX: no longer names the net of U4.56 (PD9)
- net PMM_SHDN: no longer names the net of U4.57 (PD10)
- net PMM_TX: no longer names the net of U4.55 (PD8)
- no-connect marks 8 -> 10
Other:
- moved on the sheet: C11, C8, Y1
