File: kicad/storage.kicad_sch (KiCad schematic)
At the start: 1 part, among them J4 Micro_SD_Card_Det2

Commit message: almost done schematic
Parts:
- added C43: 100nF, symbol Device:C_Small
- added R9: 10k, symbol Device:R_Small_US
Connections:
- net 3.3V: now also J4.10 (DET_A), J4.4 (VDD), C43.1
- net CARD_DETECT: now also J4.9 (DET_B), R9.1
- net GND: now also J4.6 (VSS), C43.2, R9.2

Commit message: almost done!
Parts:
- C43: footprint (none) -> Capacitor_SMD:C_0603_1608Metric
- renumbered J4 to J5
Changed lines of the file:
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@@
 		(dnp no)
 		(fields_autoplaced yes)
-		(property "Reference" "J4"
+		(property "Reference" "J5"
 			(at 123.825 46.99 0)
 			(show_name no)
@@
 			(project "MP3player"
 				(path "/c86fdb70-ebb0-4c87-946f-42a0fbefb388/719a4c5b-010e-4480-a891-7346e02ef661"
-					(reference "J4")
+					(reference "J5")
 					(unit 1)
 				)
@@
 			)
 		)
-		(property "Footprint" ""
+		(property "Footprint" "Capacitor_SMD:C_0603_1608Metric"
 			(at 76.2 68.58 0)
 			(hide yes)

Commit message: general changes
Parts:
- J5: footprint (none) -> Connector_Card:microSD_HC_Hirose_DM3D-SF
- R9: footprint (none) -> Resistor_SMD:R_0603_1608Metric
Changed lines of the file:
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@@
 			)
 		)
-		(property "Footprint" ""
+		(property "Footprint" "Connector_Card:microSD_HC_Hirose_DM3D-SF"
 			(at 175.26 50.8 0)
 			(hide yes)
@@
 			)
 		)
-		(property "Footprint" ""
+		(property "Footprint" "Resistor_SMD:R_0603_1608Metric"
 			(at 100.33 88.9 0)
 			(hide yes)
