File: kicad/vcp_filt.kicad_sch (KiCad schematic)
At the start: 5 parts

Commit message: almost done!
Parts:
- C130, C131, C132, C133, C134: footprint (none) -> Capacitor_SMD:C_0603_1608Metric
Changed lines of the file:
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@@
 			)
 		)
-		(property "Footprint" ""
+		(property "Footprint" "Capacitor_SMD:C_0603_1608Metric"
 			(at 40.64 69.85 0)
 			(hide yes)
@@
 			)
 		)
-		(property "Footprint" ""
+		(property "Footprint" "Capacitor_SMD:C_0603_1608Metric"
 			(at 50.8 54.61 0)
 			(hide yes)
@@
 			)
 		)
-		(property "Footprint" ""
+		(property "Footprint" "Capacitor_SMD:C_0603_1608Metric"
 			(at 40.64 62.23 0)
 			(hide yes)
@@
 			)
 		)
-		(property "Footprint" ""
+		(property "Footprint" "Capacitor_SMD:C_0603_1608Metric"
 			(at 40.64 54.61 0)
 			(hide yes)
@@
 			)
 		)
-		(property "Footprint" ""
+		(property "Footprint" "Capacitor_SMD:C_0603_1608Metric"
 			(at 60.96 54.61 0)
 			(hide yes)

Commit message: general changes
Parts:
- renumbered C130 to C54, C131 to C55, C132 to C56, C133 to C57, C134 to C58
Changed lines of the file:
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@@
 		(dnp no)
 		(fields_autoplaced yes)
-		(property "Reference" "C132"
+		(property "Reference" "C56"
 			(at 43.18 68.5862 0)
 			(show_name no)
@@
 			(project "MP3player"
 				(path "/c86fdb70-ebb0-4c87-946f-42a0fbefb388/8ec0c330-8240-4e36-aed2-8b84a8e7f410/fae2aa14-d6a3-4ea7-96f8-e52515107470"
-					(reference "C132")
+					(reference "C56")
 					(unit 1)
 				)
@@
 		(dnp no)
 		(fields_autoplaced yes)
-		(property "Reference" "C133"
+		(property "Reference" "C57"
 			(at 53.34 53.3462 0)
 			(show_name no)
@@
 			(project "MP3player"
 				(path "/c86fdb70-ebb0-4c87-946f-42a0fbefb388/8ec0c330-8240-4e36-aed2-8b84a8e7f410/fae2aa14-d6a3-4ea7-96f8-e52515107470"
-					(reference "C133")
+					(reference "C57")
 					(unit 1)
 				)
@@
 		(dnp no)
 		(fields_autoplaced yes)
-		(property "Reference" "C131"
+		(property "Reference" "C55"
 			(at 43.18 60.9662 0)
 			(show_name no)
@@
 			(project "MP3player"
 				(path "/c86fdb70-ebb0-4c87-946f-42a0fbefb388/8ec0c330-8240-4e36-aed2-8b84a8e7f410/fae2aa14-d6a3-4ea7-96f8-e52515107470"
-					(reference "C131")
+					(reference "C55")
 					(unit 1)
 				)
@@
 		(dnp no)
 		(fields_autoplaced yes)
-		(property "Reference" "C130"
+		(property "Reference" "C54"
 			(at 43.18 53.3462 0)
 			(show_name no)
@@
 			(project "MP3player"
 				(path "/c86fdb70-ebb0-4c87-946f-42a0fbefb388/8ec0c330-8240-4e36-aed2-8b84a8e7f410/fae2aa14-d6a3-4ea7-96f8-e52515107470"
-					(reference "C130")
+					(reference "C54")
 					(unit 1)
 				)
@@
 		(dnp no)
 		(fields_autoplaced yes)
-		(property "Reference" "C134"
+		(property "Reference" "C58"
 			(at 63.5 53.3462 0)
 			(show_name no)
@@
 			(project "MP3player"
 				(path "/c86fdb70-ebb0-4c87-946f-42a0fbefb388/8ec0c330-8240-4e36-aed2-8b84a8e7f410/fae2aa14-d6a3-4ea7-96f8-e52515107470"
-					(reference "C134")
-					(unit 1)
-				)
+					(reference "C58")
+					(unit 1)
+				)
