File: kicad/_restore_backup_2026-06-30T12-19-51-104/microphone.kicad_sch (KiCad schematic)
At the start: 2 parts

Commit message: updates
Parts:
- renumbered C130 to C45
Other:
- moved on the sheet: C45, MK1
Changed lines of the file:
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@@
 	(paper "A4")
 	(junction
-		(at 44.45 20.32)
+		(at 39.37 27.94)
 		(diameter 0)
 		(color 0 0 0 0)
@@
 	(wire
 		(pts
-			(xy 44.45 17.78) (xy 44.45 20.32)
-		)
-		(stroke
-			(width 0)
-			(type default)
-		)
-	)
-	(wire
-		(pts
-			(xy 35.56 26.67) (xy 35.56 27.94)
-		)
-		(stroke
-			(width 0)
-			(type default)
-		)
-	)
-	(wire
-		(pts
-			(xy 54.61 39.37) (xy 55.88 39.37)
-		)
-		(stroke
-			(width 0)
-			(type default)
-		)
-	)
-	(wire
-		(pts
-			(xy 33.02 36.83) (xy 34.29 36.83)
-		)
-		(stroke
-			(width 0)
-			(type default)
-		)
-	)
-	(wire
-		(pts
-			(xy 44.45 46.99) (xy 44.45 48.26)
-		)
-		(stroke
-			(width 0)
-			(type default)
-		)
-	)
-	(wire
-		(pts
-			(xy 44.45 20.32) (xy 44.45 31.75)
-		)
-		(stroke
-			(width 0)
-			(type default)
-		)
-	)
-	(wire
-		(pts
-			(xy 35.56 21.59) (xy 35.56 20.32)
-		)
-		(stroke
-			(width 0)
-			(type default)
-		)
-	)
-	(wire
-		(pts
-			(xy 54.61 41.91) (xy 55.88 41.91)
-		)
-		(stroke
-			(width 0)
-			(type default)
-		)
-	)
-	(wire
-		(pts
-			(xy 35.56 20.32) (xy 44.45 20.32)
-		)
-		(stroke
-			(width 0)
-			(type default)
-		)
-	)
-	(wire
-		(pts
-			(xy 54.61 36.83) (xy 55.88 36.83)
-		)
-		(stroke
-			(width 0)
-			(type default)
-		)
-	)
-	(wire
-		(pts
-			(xy 43.18 17.78) (xy 44.45 17.78)
+			(xy 39.37 25.4) (xy 39.37 27.94)
+		)
+		(stroke
+			(width 0)
+			(type default)
+		)
+	)
+	(wire
+		(pts
+			(xy 30.48 34.29) (xy 30.48 35.56)
+		)
+		(stroke
+			(width 0)
+			(type default)
+		)
+	)
+	(wire
+		(pts
+			(xy 49.53 46.99) (xy 50.8 46.99)
+		)
+		(stroke
+			(width 0)
+			(type default)
+		)
+	)
+	(wire
+		(pts
+			(xy 27.94 44.45) (xy 29.21 44.45)
+		)
+		(stroke
+			(width 0)
+			(type default)
+		)
+	)
+	(wire
+		(pts
+			(xy 39.37 54.61) (xy 39.37 55.88)
+		)
+		(stroke
+			(width 0)
+			(type default)
+		)
+	)
+	(wire
+		(pts
+			(xy 39.37 27.94) (xy 39.37 39.37)
+		)
+		(stroke
+			(width 0)
+			(type default)
+		)
+	)
+	(wire
+		(pts
+			(xy 30.48 29.21) (xy 30.48 27.94)
+		)
+		(stroke
+			(width 0)
+			(type default)
+		)
+	)
+	(wire
+		(pts
+			(xy 49.53 49.53) (xy 50.8 49.53)
+		)
+		(stroke
+			(width 0)
+			(type default)
+		)
+	)
+	(wire
+		(pts
+			(xy 30.48 27.94) (xy 39.37 27.94)
+		)
+		(stroke
+			(width 0)
+			(type default)
+		)
+	)
+	(wire
+		(pts
+			(xy 49.53 44.45) (xy 50.8 44.45)
+		)
+		(stroke
+			(width 0)
+			(type default)
+		)
+	)
+	(wire
+		(pts
+			(xy 38.1 25.4) (xy 39.37 25.4)
 		)
 		(stroke
@@
 	(hierarchical_label "3.3V"
 		(shape input)
-		(at 43.18 17.78 180)
+		(at 38.1 25.4 180)
 		(effects
 			(font
@@
 	(hierarchical_label "MIC_DATA"
 		(shape input)
-		(at 55.88 41.91 0)
+		(at 50.8 49.53 0)
 		(effects
 			(font
@@
 	(hierarchical_label "MIC_LRCLK"
 		(shape input)
-		(at 55.88 36.83 0)
+		(at 50.8 44.45 0)
 		(effects
 			(font
@@
 	(hierarchical_label "MIC_CHANNEL"
 		(shape input)
-		(at 33.02 36.83 180)
+		(at 27.94 44.45 180)
 		(effects
 			(font
@@
 	(hierarchical_label "MIC_BCLK"
 		(shape input)
-		(at 55.88 39.37 0)
+		(at 50.8 46.99 0)
 		(effects
 			(font
@@
 	(symbol
 		(lib_id "Sensor_Audio:ICS-43434")
-		(at 44.45 39.37 0)
+		(at 39.37 46.99 0)
 		(unit 1)
 		(body_style 1)
@@
 		(fields_autoplaced yes)
 		(property "Reference" "MK1"
-			(at 46.5933 29.21 0)
+			(at 41.5133 36.83 0)
 			(show_name no)
 			(do_not_autoplace no)
@@
 		)
 		(property "Value" "ICS-43434"
-			(at 46.5933 31.75 0)
+			(at 41.5133 39.37 0)
 			(show_name no)
 			(do_not_autoplace no)
@@
 		)
 		(property "Footprint" "Sensor_Audio:InvenSense_ICS-43434-6_3.5x2.65mm"
-			(at 44.45 39.37 0)
+			(at 39.37 46.99 0)
 			(hide yes)
 			(show_name no)
@@
 		)
 		(property "Datasheet" "https://www.invensense.com/wp-content/uploads/2016/02/DS-000069-ICS-43434-v1.2.pdf"
-			(at 44.45 39.37 0)
+			(at 39.37 46.99 0)
 			(hide yes)
 			(show_name no)
@@
 		)
 		(property "Description" "TDK InvenSense MEMS Microphone, 24-bit I2S, 65 dBA SNR, LGA-6"
-			(at 44.45 39.37 0)
+			(at 39.37 46.99 0)
 			(hide yes)
 			(show_name no)
@@
 	(symbol
 		(lib_id "Device:C_Small")
-		(at 35.56 24.13 0)
+		(at 30.48 31.75 0)
 		(unit 1)
 		(body_style 1)
@@
 		(dnp no)
 		(fields_autoplaced yes)
-		(property "Reference" "C130"
-			(at 38.1 22.8662 0)
+		(property "Reference" "C45"
+			(at 33.02 30.4862 0)
 			(show_name no)
 			(do_not_autoplace no)
@@
 		)
 		(property "Value" "100nF"
-			(at 38.1 25.4062 0)
+			(at 33.02 33.0262 0)
 			(show_name no)
 			(do_not_autoplace no)
@@
 		)
 		(property "Footprint" ""
-			(at 35.56 24.13 0)
+			(at 30.48 31.75 0)
 			(hide yes)
 			(show_name no)
@@
 		)
 		(property "Datasheet" ""
-			(at 35.56 24.13 0)
+			(at 30.48 31.75 0)
 			(hide yes)
 			(show_name no)
@@
 		)
 		(property "Description" "Unpolarized capacitor, small symbol"
-			(at 35.56 24.13 0)
+			(at 30.48 31.75 0)
 			(hide yes)
 			(show_name no)
@@
 			(project "MP3player"
 				(path "/c86fdb70-ebb0-4c87-946f-42a0fbefb388/3c7a344c-7f88-4b5c-bff2-9cbba23de578"
-					(reference "C130")
+					(reference "C45")
 					(unit 1)
 				)
@@
 	(symbol
 		(lib_id "power:GND")
-		(at 44.45 48.26 0)
+		(at 39.37 55.88 0)
 		(unit 1)
 		(body_style 1)
@@
 		(dnp no)
 		(fields_autoplaced yes)
-		(property "Reference" "#PWR047"
-			(at 44.45 54.61 0)
+		(property "Reference" "#PWR042"
+			(at 39.37 62.23 0)
 			(hide yes)
 			(show_name no)
@@
 		)
 		(property "Value" "GND"
-			(at 44.45 53.34 0)
+			(at 39.37 60.96 0)
 			(show_name no)
 			(do_not_autoplace no)
@@
 		)
 		(property "Footprint" ""
-			(at 44.45 48.26 0)
+			(at 39.37 55.88 0)
 			(hide yes)
 			(show_name no)
@@
 		)
 		(property "Datasheet" ""
-			(at 44.45 48.26 0)
+			(at 39.37 55.88 0)
 			(hide yes)
 			(show_name no)
@@
 		)
 		(property "Description" "Power symbol creates a global label with name \"GND\" , ground"
-			(at 44.45 48.26 0)
+			(at 39.37 55.88 0)
 			(hide yes)
 			(show_name no)
@@
 			(project "MP3player"
 				(path "/c86fdb70-ebb0-4c87-946f-42a0fbefb388/3c7a344c-7f88-4b5c-bff2-9cbba23de578"
-					(reference "#PWR047")
+					(reference "#PWR042")
 					(unit 1)
 				)
@@
 	(symbol
 		(lib_id "power:GND")
-		(at 35.56 27.94 0)
+		(at 30.48 35.56 0)
 		(unit 1)
 		(body_style 1)
@@
 		(dnp no)
 		(fields_autoplaced yes)
-		(property "Reference" "#PWR046"
-			(at 35.56 34.29 0)
+		(property "Reference" "#PWR045"
+			(at 30.48 41.91 0)
 			(hide yes)
 			(show_name no)
@@
 		)
 		(property "Value" "GND"
-			(at 35.56 33.02 0)
+			(at 30.48 40.64 0)
 			(show_name no)
 			(do_not_autoplace no)
@@
 		)
 		(property "Footprint" ""
-			(at 35.56 27.94 0)
+			(at 30.48 35.56 0)
 			(hide yes)
 			(show_name no)
@@
 		)
 		(property "Datasheet" ""
-			(at 35.56 27.94 0)
+			(at 30.48 35.56 0)
 			(hide yes)
 			(show_name no)
@@
 		)
 		(property "Description" "Power symbol creates a global label with name \"GND\" , ground"
-			(at 35.56 27.94 0)
+			(at 30.48 35.56 0)
 			(hide yes)
 			(show_name no)
@@
 			(project "MP3player"
 				(path "/c86fdb70-ebb0-4c87-946f-42a0fbefb388/3c7a344c-7f88-4b5c-bff2-9cbba23de578"
-					(reference "#PWR046")
+					(reference "#PWR045")
 					(unit 1)
 				)
