File: kicad/_restore_backup_2026-06-30T12-19-51-104/power.kicad_sch (KiCad schematic)
At the start: 66 parts, among them J1 USB_C_Receptacle_USB2.0_14P, SW1 SW_Push, SW2 SW_Push, U1 TPS628438DRL, U2 BQ25895RTW, U3 USBLC6-2SC6, U4 MAX17263xxTE, U5 TLV70233_SOT23-5, U6 TPS7A4701xRGW

Commit message: updates
Parts:
- renumbered C3 to C1, C4 to C10, C6 to C11, C20 to C12, C21 to C13, C17 to C14, C18 to C15, C23 to C16, C22 to C17, C24 to C18, C9 to C19, C5 to C2, C7 to C20, C15 to C21, C2 to C22, C1 to C23, C8 to C24, C19 to C25, C16 to C26, C11 to C3, C10 to C4, C13 to C5, C14 to C6, C12 to C7, D2 to D1, D1 to D72, D4 to D76, D5 to D77, D6 to D78, D3 to D81, L2 to L1, L1 to L2, R14 to R10, R6 to R11, R15 to R12, R16 to R13, R17 to R14, R18 to R15, R19 to R16, R21 to R17, R20 to R18, R3 to R19, R9 to R20, R10 to R21, R5 to R3, R7 to R5, R8 to R6, R11 to R7, R12 to R8, R13 to R9, U3 to U1, U1 to U4, U4 to U6, U6 to U7
Connections:
- net +3.3v_AUX renamed 3.3v_AUX
- net BQ25895_CE renamed CE
- net BQ25895_INT renamed INT_FG
- net BQ25895_OTG renamed OTG
- net MAX17263_ALRT renamed MAX_ALRT
- net PWR_I2C_SCL renamed SCL_FG
- net SCL_FG: no longer U6.14 (SCL)
- net PWR_I2C_SDA renamed SDA_FG
- net SDA_FG: no longer U6.13 (SDA)
- new net MAX_SCL: U6.14 (SCL)
- new net MAX_SDA: U6.13 (SDA)
Other:
- moved on the sheet: C26
