File: kicad/_restore_backup_2026-06-30T12-19-51-104/stm32core.kicad_sch (KiCad schematic)
At the start: 32 parts, among them J2 Conn_01x05, U7 STM32H743VIT6, U8 DS3231M, Y1 8MHz, Y2 32.768KHz

Commit message: updates
Parts:
- renumbered BT4 to BT3, BT3 to BT4, C36 to C27, C33 to C28, C32 to C29, C31 to C30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
Connections:
- net VREF: no longer names the net of U8.20 (VREF+)
