File: kicad/_restore_backup_2026-06-30T12-19-51-104/storage.kicad_sch (KiCad schematic)
At the start: 1 part, among them J4 Micro_SD_Card_Det2

Commit message: updates
Parts:
- renumbered J4 to J3
Changed lines of the file:
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@@
 	(hierarchical_label "CARD_DETECT"
 		(shape input)
-		(at 77.47 81.28 180)
-		(effects
-			(font
-				(size 1.27 1.27)
-			)
-			(justify right)
+		(at 38.1 25.4 0)
+		(effects
+			(font
+				(size 1.27 1.27)
+			)
+			(justify left)
 		)
 	)
@@
 		(dnp no)
 		(fields_autoplaced yes)
-		(property "Reference" "J4"
+		(property "Reference" "J3"
 			(at 123.825 46.99 0)
 			(show_name no)
@@
 			(project "MP3player"
 				(path "/c86fdb70-ebb0-4c87-946f-42a0fbefb388/719a4c5b-010e-4480-a891-7346e02ef661"
-					(reference "J4")
+					(reference "J3")
 					(unit 1)
 				)
@@
 		(dnp no)
 		(fields_autoplaced yes)
-		(property "Reference" "#PWR043"
+		(property "Reference" "#PWR017"
 			(at 144.78 88.9 0)
 			(hide yes)
@@
 			(project "MP3player"
 				(path "/c86fdb70-ebb0-4c87-946f-42a0fbefb388/719a4c5b-010e-4480-a891-7346e02ef661"
-					(reference "#PWR043")
+					(reference "#PWR017")
 					(unit 1)
 				)
