File: kicad/_restore_backup_2026-07-22T15-47-04-759/audio.kicad_sch (KiCad schematic)
At the start: 12 parts, among them J3 SHOU HAN PJ-342, U9 CS43131-CNZR

Commit message: almost done schematic
Parts:
- removed C34, C35, C41: 100nF, symbol Device:C_Small
- removed C36, C37: 15uF, symbol Device:C_Small
- removed C38, C39, C40: 2.2uF, symbol Device:C_Small
- removed C42: 4.7uF, symbol Device:C_Small
- removed TP3: TestPoint, symbol Connector:TestPoint
- added C137, C138: 10pF, symbol Device:C_Small
- added C139: 4.7uF, symbol Device:C_Small
- added C140, C141, C142: 0.1uF, symbol Device:C_Small
- added C45, C46, C47: 2.2uF, symbol Device:C_Small
- added Y4: 22.5792MHz, symbol Device:Crystal
Connections:
- net VCP_FILT/GNDCP is gone; now on net GND: U9.19 (GNDCP)
- net 3.3V_AUDIO: no longer U9.26 (VP)
- net GND: now also U9.41 (EP), C137.2, C138.2, C139.1, C140.1, C141.1, C142.1; no longer J3.G, J3.R2, U9.13 (HPREFA), U9.17 (HPREFB), U9.30 (ADR), U9.36 (XTO)
- net I2S_BCLK: no longer U9.34 (SCLK1)
- net I2S_LRCLK: no longer U9.38 (LRCK1)
- net I2S_MCLK: no longer U9.37 (XTI/MCLK)
- net I2S_SDOUT: no longer U9.2 (SDIN1)
- net at U9.10 (FLYP_VA): now also C47.1
- net at U9.11 (FLYN_VA): now also C47.2
- net at U9.14 (HPOUTA): no longer J3.T
- net at U9.16 (HPOUTB): no longer J3.R1
- net at U9.22 (HP_DETECT): no longer J3.TN
- removed net 1.8v: U9.31 (VL), U9.4 (VD), U9.7 (VA)
- net INT: no longer names the net of U9.27 (~{INT})
- net RESET: no longer names the net of U9.28 (~{RESET})
- net VCP_FILT/FLYC_VCP: no longer names the net of U9.23 (FLYC_VCP)
- net VCP_FILT/FLYC_VCP: now also C45.2
- net VCP_FILT/FLYN_VCP: no longer names the net of U9.20 (FLYN_VCP)
- net VCP_FILT/FLYN_VCP: now also C45.1, C46.1
- net VCP_FILT/FLYP_VCP: no longer names the net of U9.24 (FLYP_VCP)
- net VCP_FILT/FLYP_VCP: now also C46.2
- net VCP_FILT/VCP: no longer names the net of U9.25 (VCP)
- net VCP_FILT/VCP_FILT+: no longer names the net of U9.21 (VCP_FILT+)
- net VCP_FILT/VCP_FILT-: no longer names the net of U9.18 (VCP_FILT–)
- new net: C139.2, C140.2, U9.26 (VP)
- new net: C137.1, U9.37 (XTI/MCLK), Y4.1
- new net: C142.2, U9.4 (VD)
- new net: C141.2, U9.31 (VL)
- new net: C138.1, U9.36 (XTO), Y4.2
- no-connect marks 8 -> 0
Other:
- removed sheet VCP_FILT
- note added: "+VD.CSP"
- note added: "+VL.CSP"
- note added: "+VP.CSP"
- moved on the sheet: J3
