File: kicad/_restore_backup_2026-07-22T15-47-04-759/microphone.kicad_sch (KiCad schematic)
At the start: 3 parts

Commit message: almost done schematic
Parts:
- removed R20: 10k, symbol Device:R_Small_US
- renumbered C129 to C130
Other:
- moved on the sheet: C130, MK1
