File: kicad/_restore_backup_2026-07-22T15-47-04-759/power.kicad_sch (KiCad schematic)
At the start: 17 parts, among them J1 USB_C_Receptacle_USB2.0_14P, U1 USBLC6-2SC6, U2 TLV70233_SOT23-5, U3 TPS7A4701xRGW

Commit message: almost done schematic
Parts:
- BT1: footprint Battery:BatteryHolder_Keystone_1042_1x18650 -> (none)
- renumbered C1 to C17, C2 to C18, C3 to C20, C4 to C21, C5 to C22, C6 to C23, C7 to C24, R4 to R10, R1 to R5, R2 to R7, R3 to R9, U1 to U3, U2 to U5, U3 to U6
Connections:
- net GND: no longer BT1.2 (-)
- net FORCE: no longer names the net of A1.18 (FORCE_ON)
- net INIT: no longer names the net of A1.15 (PMM_INIT)
- net SCL: no longer names the net of A1.14 (SCL)
- net SDA: no longer names the net of A1.13 (SDA)
- net SHDN: no longer names the net of A1.17 (SHDN)
- net SWCLK: no longer names the net of A1.39 (SWCLK)
- net SWDIO: no longer names the net of A1.40 (SWDIO)
- net UART_RX: no longer names the net of A1.36 (UART_RX)
- net UART_TX: no longer names the net of A1.37 (UART_TX)
- net VBUS renamed USB_VBUS
- no-connect marks 23 -> 8
Other:
- moved on the sheet: BT1
