File: kicad/_restore_backup_2026-07-22T15-47-04-759/radio.kicad_sch (KiCad schematic)
At the start: 15 parts, among them J5 SMA, J6 SMA, U10 Si4735-D60-GU

Commit message: almost done schematic
Parts:
- removed J5, J6: SMA, Connector_Coaxial:SMA_Amphenol_901-143_Horizontal, symbol Connector:Conn_Coaxial_Small
- removed JP1: SolderJumper_3_Bridged12, symbol Jumper:SolderJumper_3_Bridged12
- removed R10: 10k, symbol Device:R_Small_US
- removed TP4, TP5, TP6: TestPoint, symbol Connector:TestPoint
- added C134, C135: 22pF, symbol Device:C_Small
- added C136: 2-5pF, symbol Device:C_Small
- added R27, R28: 2k, symbol Device:R_Small_US
- added Y3: 32.768KHz, symbol Device:Crystal
- L3: renamed from L1; value 450uH -> 180-450uH
- renumbered C47 to C131, C48 to C132, C46 to C133, C44 to C48, C45 to C49, R11 to R26
Connections:
- net GND: now also C134.2, C135.2, C136.2; no longer L3.2, U10.9 (RFGND)
- net RADIO_RST: no longer U10.15 (~{RST})
- net RADIO_SCL: no longer U10.17 (SCLK)
- net RADIO_SDA: no longer U10.18 (SDIO)
- net SEN: now reaches U10.16 (~{SEN})
- net at U10.19 (RCLK): now also C135.1, Y3.1
- net ROUT: now reaches U10.23 (ROUT/[DOUT])
- net LOUT: now reaches U10.24 (LOUT/[DFS])
- net DFS: now reaches C133.2, L3.1
- net DFS: now also C136.1, R27.2
- net RADIO_I2S_BCLK: no longer names the net of U10.3 (GPO3/[DCLK])
- net RADIO_I2S_BCLK: now also R28.2
- net RADIO_I2S_DATA renamed DOUT
- net RADIO_I2S_LRCLK: no longer names the net of U10.2 (DFS)
- net RADIO_I2S_LRCLK: now also R27.1
- new net: L3.2, U10.9 (RFGND)
- new net: C134.1, R28.1, Y3.2
- new net RST: U10.15 (~{RST})
- new net SCLK: U10.17 (SCLK)
- new net SDIO: U10.18 (SDIO)
Other:
- moved on the sheet: L3, R26
