File: kicad/_restore_backup_2026-07-22T15-47-04-759/sparkles.kicad_sch (KiCad schematic)
At the start: 160 parts

Commit message: almost done schematic
Parts:
- renumbered C99 to C100, C100 to C101, C101 to C102, C102 to C103, C103 to C104, C104 to C105, C105 to C106, C106 to C107, C107 to C108, C108 to C109, C109 to C110, C110 to C111, C111 to C112, C112 to C113, C113 to C114, C114 to C115, C115 to C116, C116 to C117, C117 to C118, C118 to C119, C119 to C120, C120 to C121, C121 to C122, C122 to C123, C123 to C124, C124 to C125, C125 to C126, C126 to C127, C127 to C128, C128 to C129, C49 to C50, C50 to C51, C51 to C52, C52 to C53, C53 to C54, C54 to C55, C55 to C56, C56 to C57, C57 to C58, C58 to C59, C59 to C60, C60 to C61, C61 to C62, C62 to C63, C63 to C64, C64 to C65, C65 to C66, C66 to C67, C67 to C68, C68 to C69, C69 to C70, C70 to C71, C71 to C72, C72 to C73, C73 to C74, C74 to C75, C75 to C76, C76 to C77, C77 to C78, C78 to C79, C79 to C80, C80 to C81, C81 to C82, C82 to C83, C83 to C84, C84 to C85, C85 to C86, C86 to C87, C87 to C88, C88 to C89, C89 to C90, C90 to C91, C91 to C92, C92 to C93, C93 to C94, C94 to C95, C95 to C96, C96 to C97, C97 to C98, C98 to C99, D7 to D10, D8 to D11, D9 to D12, D10 to D13, D11 to D14, D12 to D15, D13 to D16, D14 to D17, D15 to D18, D16 to D19, D17 to D20, D18 to D21, D19 to D22, D20 to D23, D21 to D24, D22 to D25, D23 to D26, D24 to D27, D25 to D28, D26 to D29, D27 to D30, D28 to D31, D29 to D32, D30 to D33, D31 to D34, D32 to D35, D33 to D36, D34 to D37, D35 to D38, D36 to D39, D37 to D40, D38 to D41, D39 to D42, D40 to D43, D41 to D44, D42 to D45, D43 to D46, D44 to D47, D45 to D48, D46 to D49, D47 to D50, D48 to D51, D49 to D52, D50 to D53, D51 to D54, D52 to D55, D53 to D56, D54 to D57, D55 to D58, D56 to D59, D57 to D60, D58 to D61, D59 to D62, D60 to D63, D61 to D64, D62 to D65, D63 to D66, D64 to D67, D65 to D68, D66 to D69, D4 to D7, D67 to D70, D68 to D71, D69 to D72, D70 to D73, D71 to D74, D72 to D75, D73 to D76, D74 to D77, D75 to D78, D76 to D79, D5 to D8, D77 to D80, D78 to D81, D79 to D82, D80 to D83, D81 to D84, D82 to D85, D83 to D86, D6 to D9
