File: kicad/_restore_backup_2026-07-28T17-16-35-996/MP3player.kicad_pcb (KiCad board)
At the start: 6 copper layers, 50 x 70 mm, 148 parts, among them J1 USB_C_Receptacle_USB2.0_14P, J2 Conn_01x02, J3 Conn_01x05, J4 AudioJack3_Ground_SwitchTR, J5 Micro_SD_Card_Det2, J6 SMA, J7 SMA, J8 Conn_01x08, SW1 SW_Push, SW10 SW_Push, SW11 SW_Push, SW12 SW_Push, SW13 SW_Push, SW14 SW_Push, SW15 SW_Push, SW16 SW_Push, SW17 SW_Push, SW2 SW_Push, SW3 SW_Push, SW4 SW_Push, SW5 SW_Push, SW6 SW_Push, SW7 SW_Push, SW8 SW_Push, SW9 SW_Push, U1 USBLC6-2SC6, U10 Si4735-D60-GU, U11 BQ24090DGQ, U12 TPS613222ADBV, U2 TLV70233_SOT23-5, U3 TPS7A4701xRGW, U4 STM32H743VIT6, U5 ISL29035, U6 LSM6DSL, U7 DS3231M, U8 BME680, U9 CS43131-CNZR, Y1 8MHz TXC AA08000002

Commit message: fininshed pcb and fixed drc errors
Routing:
- net /OLED UI/Row1: track 82.7 -> 20.8 mm, vias 4 -> 2
- net /OLED UI/Row2: track 69.6 -> 21.5 mm
- net /OLED UI/BTN_BOOT0: track 46.9 -> 9.75 mm, vias 2 -> 0
- net +3.3V: track 181.1 -> 145.5 mm, vias 24 -> 22
- net /OLED UI/Row3: track 49.3 -> 17.8 mm
- net /OLED UI/BTN_RST: track 64.5 -> 37.6 mm
- net GND: track 251.3 -> 224.5 mm, vias 56 -> 54
- net /Radio/RADIO_RST: track 25.1 -> 3.29 mm, vias 2 -> 1
- net /Radio/RADIO_SCL: track 25.3 -> 4.08 mm, vias 2 -> 1
- net Net-(JP1-B): track 12.3 -> 0.00 mm
- net /Radio/RADIO_SDA: track 14.8 -> 3.09 mm, vias 2 -> 1
- net Net-(U10-LOUT/[DFS]): track 22.2 -> 17.2 mm
- net SENSORS_SPI1_MOSI: track 34.1 -> 36.5 mm
- net /OLED UI/BTN_LOCK: track 57.5 -> 55.3 mm
- net /OLED UI/OLED_BL: track 11.5 -> 9.67 mm
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